File: ADRmu.kicad_pcb (KiCad board)
At the start: 2 copper layers, 160 x 100 mm, 34 parts, among them J1 DIN41612_02x16_AC_EvenPins, J10 Conn_01x01, J2 Conn_01x01, J3 Conn_01x01, J4 Conn_01x01, J5 Conn_01x01, J6 Conn_01x01, J7 Conn_01x01, J8 Conn_01x01, J9 Conn_01x01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

Commit message: asdf
Parts:
- added D3: D, Diode_SMD:D_SOD-123, F.Cu at (111.8, 73.7)
- added D4: D, Diode_SMD:D_SOD-123, F.Cu at (111.8, 70.3)
- added J11: Conn_01x01, Connector_Wire:SolderWire-1sqmm_1x01_D1.4mm_OD3.9mm, F.Cu at (182.9, 73.7)
- added J12: Conn_01x01, Connector_Wire:SolderWire-1sqmm_1x01_D1.4mm_OD3.9mm, F.Cu at (167.6, 73.7)
- added Q1: Q_NPN_BCE, Package_TO_SOT_SMD:SOT-223-3_TabPin2, F.Cu at (104.0, 72.8)
- added RN1: 322146, Package_DIP:DIP-14_W7.62mm, F.Cu at (25.2, 98.2)
- added U5: Opamp_Dual, Package_SO:SOIC-8_3.9x4.9mm_P1.27mm, F.Cu at (38.7, 99.3)
- moved J9 37.6 mm to (167.6, 129.5)
- moved J10 33.6 mm to (188.0, 129.5)
- moved J8 30.7 mm to (177.8, 129.5)
Connections:
- U4 pad 1: unconnected-(U4-Pad1) -> Net-(U4-Pad1)
- U4 pad 2: unconnected-(U4-Pad2) -> Net-(U4-Pad2)
- U4 pad 3: unconnected-(U4-Pad3) -> Net-(U4-Pad3)
- U4 pad 4: unconnected-(U4-Pad4) -> Net-(U4-Pad4)
- U4 pad 5: unconnected-(U4-Pad5) -> Net-(U4-Pad5)
- U4 pad 6: unconnected-(U4-Pad6) -> Net-(U4-Pad6)
- U4 pad 7: unconnected-(U4-Pad7) -> Net-(U4-Pad7)
- U4 pad 8: unconnected-(U4-Pad8) -> Net-(U4-Pad8)
Other:
- copper layers 2 -> 4

Commit message: asdf
Parts:
- added C7: 100n, Capacitor_SMD:C_0805_2012Metric, F.Cu at (45.7, 55.9)
- added C8: 100n, Capacitor_SMD:C_0805_2012Metric, F.Cu at (54.2, 49.4)
- added R7: 1k, Resistor_SMD:R_0805_2012Metric, F.Cu at (54.1, 52.4)
- added R8: 1M, Resistor_SMD:R_0805_2012Metric, F.Cu at (45.7, 58.9)
- added R9: 10k, Resistor_SMD:R_0805_2012Metric, F.Cu at (50.1, 55.9)
- moved U5 49.0 mm to (47.7, 51.1)
- moved RN1 49.0 mm to (34.3, 50.0)
Connections:
- D3 pad 1: unconnected-(D3-Pad1) -> /ref/GNDf
- Q1 pad 1: unconnected-(Q1-Pad1) -> Net-(Q1-Pad1)
- Q1 pad 2: unconnected-(Q1-Pad2) -> /ref/12Vf
- RN1 pad 11: Net-(U4-Pad6) -> /ref/ADR_Pin6
- RN1 pad 12: Net-(U4-Pad7) -> Net-(C8-Pad1)
- RN1 pad 13: Net-(U4-Pad5) -> /ref/ADR_Pin8
- RN1 pad 14: Net-(U4-Pad8) -> Net-(RN1-Pad14)
- RN1 pad 4: Net-(U4-Pad7) -> /ref/ADR_Pin6
- RN1 pad 7: unconnected-(RN1-Pad7) -> Net-(RN1-Pad7)
- RN1 pad 9: unconnected-(RN1-Pad9) -> Net-(RN1-Pad7)
- U4 pad 5: Net-(U4-Pad5) -> Net-(RN1-Pad14)
- U4 pad 6: Net-(U4-Pad6) -> /ref/ADR_Pin6
- U4 pad 7: Net-(U4-Pad7) -> Net-(C8-Pad1)
- U4 pad 8: Net-(U4-Pad8) -> /ref/ADR_Pin8
- U5 pad 5: unconnected-(U5-Pad5) -> /ref/ADR_Pin8
- U5 pad 6: unconnected-(U5-Pad6) -> Net-(R8-Pad2)
- U5 pad 7: unconnected-(U5-Pad7) -> Net-(R7-Pad2)
Routing:
- net Net-(D4-Pad1): track 0.00 -> 2.54 mm

Commit message: asdf
Parts:
- added C10: 100n, Capacitor_SMD:C_0805_2012Metric, F.Cu at (51.4, 91.4)
- added C9: 100n, Capacitor_SMD:C_0805_2012Metric, F.Cu at (55.9, 91.4)
- moved RN1 118.1 mm to (103.4, 145.8), turned to 90 degrees
- moved Q1 19.8 mm to (114.3, 55.9)
- moved U4 4.18 mm to (110.0, 97.1), turned to -90 degrees
Connections:
- net Net-(D4-Pad1) renamed /ref/ADR_Pin3
- C8 pad 1: Net-(C8-Pad1) -> /ref/ADR_Pin7
- D4 pad 2: unconnected-(D4-Pad2) -> Net-(C10-Pad1)
- RN1 pad 12: Net-(C8-Pad1) -> /ref/ADR_Pin7
- RN1 pad 14: Net-(RN1-Pad14) -> /ref/ADR_Pin5
- RN1 pad 3: Net-(RN1-Pad3) -> /ref/ADR_Pin4
- RN1 pad 4: /ref/ADR_Pin6 -> /ref/ADR_Pin7
- RN1 pad 7: Net-(RN1-Pad7) -> unconnected-(RN1-Pad7)
- RN1 pad 9: Net-(RN1-Pad7) -> Net-(RN1-Pad9)
- U4 pad 4: Net-(RN1-Pad3) -> /ref/ADR_Pin4
- U4 pad 5: Net-(RN1-Pad14) -> /ref/ADR_Pin5
- U4 pad 7: Net-(C8-Pad1) -> /ref/ADR_Pin7
- U5 pad 1: unconnected-(U5-Pad1) -> Net-(C10-Pad1)
- U5 pad 2: unconnected-(U5-Pad2) -> /ref/ADR_Pin4
- U5 pad 3: unconnected-(U5-Pad3) -> /ref/ADR_Pin5
Routing:
- net Net-(D3-Pad2): track 0.00 -> 33.8 mm
- net /ref/ADR_Pin8: track 0.00 -> 33.8 mm
- net /ref/ADR_Pin6: track 0.00 -> 33.7 mm
- net /ref/ADR_Pin4: track 0.00 -> 33.7 mm
- net Net-(C7-Pad1): track 0.00 -> 32.2 mm
- net /ref/ADR_Pin7: track 0.00 -> 32.1 mm
- net /ref/ADR_Pin5: track 0.00 -> 32.1 mm
- net /ref/ADR_Pin3: track 2.54 -> 34.7 mm

Commit message: asdf
Parts:
- added H1: MountingHole, MountingHole:MountingHole_4.3mm_M4, F.Cu at (157.0, 82.0)
- added H2: MountingHole, MountingHole:MountingHole_4.3mm_M4, F.Cu at (170.0, 95.0)
- added H3: MountingHole, MountingHole:MountingHole_4.3mm_M4, F.Cu at (193.0, 82.0)
- added H4: MountingHole, MountingHole:MountingHole_4.3mm_M4, F.Cu at (180.0, 95.0)
- added H5: MountingHole, MountingHole:MountingHole_4.3mm_M4, F.Cu at (193.0, 118.0)
- added H6: MountingHole, MountingHole:MountingHole_4.3mm_M4, F.Cu at (180.0, 105.0)
- added H7: MountingHole, MountingHole:MountingHole_4.3mm_M4, F.Cu at (157.0, 118.0)
- added H8: MountingHole, MountingHole:MountingHole_4.3mm_M4, F.Cu at (170.0, 105.0)
- moved C1 102.3 mm to (209.0, 62.0), turned to -90 degrees
- moved U2 65.5 mm to (134.0, 161.0)
- moved C4 56.3 mm to (137.0, 166.0)
- moved U1 55.6 mm to (143.0, 162.0)
- moved R1 55.2 mm to (140.0, 171.0)
- moved R2 49.8 mm to (150.0, 168.0)
- moved JP3 44.3 mm to (144.7, 156.0)
- moved R3 43.8 mm to (145.1, 169.0)
- moved JP2 43.5 mm to (150.0, 162.0)
- moved JP1 43.2 mm to (150.3, 159.0)
- moved JP4 37.6 mm to (151.3, 156.0)
- moved R5 16.8 mm to (180.1, 155.0)
- moved C6 16.4 mm to (181.1, 160.0)
- moved R4 14.0 mm to (175.0, 159.0)
- moved C5 9.68 mm to (172.1, 167.0)
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Routing:
- net GND: track 15.2 -> 26.4 mm
- net +12V: track 5.08 -> 16.2 mm
- net /ref/ADR_Pin3: track 34.7 -> 32.1 mm

Commit message: asdf
Parts:
- removed D1 (x2): LED, LED_SMD:LED_1206_3216Metric
- removed the D2 at (72.5, 53.5)
- moved U3 105.5 mm to (175.0, 61.0)
- moved J10 63.2 mm to (165.0, 70.0), turned to 0 degrees
- moved J11 63.2 mm to (165.0, 130.0), turned to 180 degrees
- moved J12 63.2 mm to (185.0, 130.0), turned to 180 degrees
- moved J9 63.2 mm to (185.0, 70.0), turned to 0 degrees
- moved J8 60.0 mm to (175.0, 70.0), turned to 0 degrees
- moved H1 50.9 mm to (193.0, 118.0), turned to 180 degrees
- moved H3 50.9 mm to (157.0, 118.0), turned to 180 degrees
- moved H5 50.9 mm to (157.0, 82.0), turned to 180 degrees
- moved H7 50.9 mm to (193.0, 82.0), turned to 180 degrees
- moved H2 14.1 mm to (180.0, 105.0), turned to 180 degrees
- moved H4 14.1 mm to (170.0, 105.0), turned to 180 degrees
- moved H6 14.1 mm to (170.0, 95.0), turned to 180 degrees
- moved H8 14.1 mm to (180.0, 95.0), turned to 180 degrees
Routing:
- net Net-(J9-Pad1): track 0.00 -> 11.4 mm
- net Net-(J10-Pad1): track 0.00 -> 11.4 mm

Commit message: asdf
Parts:
- added C11: 22u, Capacitor_SMD:C_1206_3216Metric, F.Cu at (95.0, 170.0)
- added C12: 22u, Capacitor_SMD:C_1206_3216Metric, F.Cu at (79.2, 180.3)
- added C13: 22u, Capacitor_SMD:C_1206_3216Metric, F.Cu at (84.8, 180.3)
- added C14: 100n, Capacitor_SMD:C_0805_2012Metric, F.Cu at (89.9, 180.1)
- added D1: LED, LED_SMD:LED_1206_3216Metric, F.Cu at (102.3, 164.5)
- added D2: D_Schottky, Diode_SMD:D_SOD-123F, F.Cu at (94.9, 173.3)
- added D5: D_Schottky, Diode_SMD:D_SOD-123F, F.Cu at (94.9, 176.7)
- added D6: D_Schottky, Diode_SMD:D_SOD-123F, F.Cu at (100.6, 170.0)
- added D7: D_Schottky, Diode_SMD:D_SOD-123F, F.Cu at (107.9, 164.4)
- added FL1: Choke_Schaffner_RN102-0.3-02-12M, Inductor_THT:Choke_Schaffner_RN102-04-14.0x14.0mm, F.Cu at (79.4, 165.8)
- added R10: 5k, Resistor_SMD:R_0805_2012Metric, F.Cu at (99.9, 173.2)
- added U6: LT3045xMSE, Package_SO:MSOP-12-1EP_3x4mm_P0.65mm_EP1.65x2.85mm, F.Cu at (95.0, 160.0)
- C3: footprint Capacitor_SMD:C_0805_2012Metric -> Capacitor_SMD:C_1206_3216Metric
- C6: value 100n -> 2.2n
- R4: value 5k -> 10k
- R5, R6: value 5k -> 16.9k
Connections:
- net /DC-DC/fault renamed /fault
- J11 pad 1: /ref/12Vf -> Net-(J11-Pad1)
- J12 pad 1: /ref/GNDf -> Net-(J12-Pad1)

Commit message: asdf
Parts:
- removed C13: 22u, Capacitor_SMD:C_1206_3216Metric
- removed the D2 at (198.3, 165.2)
- removed FL1: Choke_Schaffner_RN102-0.3-02-12M, Inductor_THT:Choke_Schaffner_RN102-04-14.0x14.0mm
- added C15: 100n, Capacitor_SMD:C_0805_2012Metric, F.Cu at (79.7, 180.6)
- added R11: 1k, Resistor_SMD:R_0805_2012Metric, F.Cu at (91.4, 169.0)
- added R12: 121k, Resistor_SMD:R_0805_2012Metric, F.Cu at (84.6, 175.4)
- moved C7 142.0 mm to (114.2, 180.3)
- moved U5 141.2 mm to (107.8, 179.0)
- moved R7 139.1 mm to (118.7, 175.7)
- moved R8 138.6 mm to (125.8, 171.9)
- moved C8 137.2 mm to (121.4, 169.0)
- moved R9 136.1 mm to (125.8, 169.0)
- moved C11 130.4 mm to (175.0, 67.0), turned to 180 degrees
- moved Q1 115.9 mm to (108.5, 171.6)
- moved C3 112.8 mm to (74.7, 180.8), turned to 0 degrees
- moved C2 112.1 mm to (87.0, 169.0), turned to 0 degrees
- moved C5 107.0 mm to (170.0, 60.0), turned to 90 degrees
- moved C10 106.3 mm to (114.2, 177.2)
- moved C9 103.8 mm to (121.4, 172.0)
- moved C12 103.3 mm to (171.0, 133.0), turned to 180 degrees
- moved C6 102.1 mm to (181.9, 57.9), turned to 90 degrees
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Connections:
- C12 pad 1: Net-(C12-Pad1) -> Net-(C14-Pad1)
- C12 pad 2: Net-(C12-Pad2) -> Net-(C14-Pad2)
- C14 pad 1: Net-(C13-Pad1) -> Net-(C14-Pad1)
- C14 pad 2: Net-(C13-Pad2) -> Net-(C14-Pad2)
- D2 pad 1: Net-(C12-Pad1) -> Net-(C14-Pad1)
- D5 pad 2: Net-(C12-Pad2) -> Net-(C14-Pad2)
- D6 pad 1: Net-(C12-Pad1) -> Net-(C14-Pad1)
- D7 pad 2: Net-(C12-Pad2) -> Net-(C14-Pad2)
- U6 pad 1: Net-(U6-Pad1) -> Net-(C14-Pad1)
- U6 pad 10: unconnected-(U6-Pad10) -> Net-(U6-Pad10)
- U6 pad 11: Net-(U6-Pad11) -> Net-(U6-Pad10)
- U6 pad 12: Net-(U6-Pad11) -> Net-(U6-Pad10)
- U6 pad 13: Net-(U6-Pad13) -> Net-(C14-Pad2)
- U6 pad 2: Net-(U6-Pad1) -> Net-(C14-Pad1)
- U6 pad 3: Net-(U6-Pad1) -> Net-(C14-Pad1)
- U6 pad 4: Net-(U6-Pad1) -> Net-(C14-Pad1)
- U6 pad 6: unconnected-(U6-Pad6) -> Net-(U6-Pad6)
- U6 pad 8: unconnected-(U6-Pad8) -> Net-(U6-Pad8)
- U6 pad 9: Net-(U6-Pad13) -> Net-(C14-Pad2)
Routing:
- net /DC-DC/sync: track 5.08 -> 57.9 mm
- net Net-(C14-Pad2): track 0.00 -> 14.1 mm
- net Net-(D6-Pad2): track 0.00 -> 8.99 mm
- net Net-(D2-Pad2): track 0.00 -> 8.99 mm
- net Net-(C14-Pad1): track 0.00 -> 6.82 mm
- net Net-(R6-Pad1): track 0.00 -> 5.20 mm
- net +12V: track 16.2 -> 20.8 mm, vias 0 -> 4
- net Net-(C6-Pad1): track 0.00 -> 4.57 mm
- net GND: track 26.4 -> 22.4 mm, vias 0 -> 10
- net Net-(R5-Pad1): track 0.00 -> 2.29 mm
- added copper zone on B.Cu, net (none)
- added copper zone on F.Cu, net (none)
- added copper zone on In1.Cu, net (none)
- added copper zone on In2.Cu, net (none)
- added copper zone on F.Cu, net +12V
- added copper zone on In1.Cu, net +12V
- added copper zone on In2.Cu, net +12V
- added copper zone on B.Cu, net GND
- added copper zone on F.Cu, net GND
- added copper zone on In1.Cu, net GND
- added copper zone on In2.Cu, net GND

Commit message: asdf
Parts:
- added C13: 100n, Capacitor_SMD:C_0805_2012Metric, F.Cu at (104.1, 70.6)
- added D8: LED, LED_SMD:LED_1206_3216Metric, F.Cu at (73.7, 67.6)
- J2: value Conn_01x01 -> 10Vf
- J3: value Conn_01x01 -> 10Vs
- J4: value Conn_01x01 -> ADRf
- J5: value Conn_01x01 -> ADRs
- J6: value Conn_01x01 -> return
- J7: value Conn_01x01 -> guard
- moved Q1 113.6 mm to (110.0, 58.0), turned to 90 degrees
- moved U5 112.6 mm to (102.1, 66.5)
- moved R7 111.2 mm to (107.7, 65.0), turned to -90 degrees
- moved D1 107.0 mm to (73.7, 62.5), turned to 90 degrees
- moved R8 104.9 mm to (107.7, 68.6), turned to 90 degrees
- moved C9 103.6 mm to (100.0, 70.6), turned to 180 degrees
- moved R9 101.7 mm to (109.7, 68.6), turned to 90 degrees
- moved D3 93.1 mm to (95.5, 81.8)
- moved D4 78.0 mm to (87.9, 96.5), turned to 180 degrees
- moved C8 77.7 mm to (131.1, 91.9), turned to 90 degrees
- moved U6 76.9 mm to (141.9, 131.6), turned to -90 degrees
- moved C14 75.9 mm to (145.5, 131.8), turned to -90 degrees
Connections:
- U5 pad 4: unconnected-(U5-Pad4) -> Net-(U5-Pad4)
- U5 pad 8: unconnected-(U5-Pad8) -> Net-(U5-Pad8)
Routing:
- net Net-(C14-Pad2): track 14.1 -> 67.7 mm
- net Net-(C14-Pad1): track 6.82 -> 54.9 mm
- net Net-(C10-Pad1): track 0.00 -> 37.8 mm
- net /ref/ADR_Pin5: track 32.1 -> 57.9 mm, vias 0 -> 1
- net Net-(C7-Pad1): track 32.2 -> 52.7 mm, vias 0 -> 1
- net /ref/ADR_Pin3: track 32.1 -> 45.3 mm, vias 0 -> 1
- net Net-(U5-Pad8): track 0.00 -> 7.79 mm
- net /ref/ADR_Pin8: track 33.8 -> 39.7 mm, vias 0 -> 1
- net Net-(U6-Pad10): track 0.00 -> 5.37 mm
- net Net-(R8-Pad2): track 0.00 -> 5.35 mm
- net /ref/ADR_Pin7: track 32.1 -> 37.1 mm, vias 0 -> 1
- net Net-(U5-Pad4): track 0.00 -> 4.45 mm
- net Net-(R7-Pad2): track 0.00 -> 3.12 mm
- net Net-(Q1-Pad1): track 0.00 -> 2.96 mm
- net Net-(D3-Pad2): track 33.8 -> 36.5 mm, vias 0 -> 1
- added copper zone on F.Cu, net /ref/12Vf
