File: ADRmu.kicad_pcb (KiCad board)
At the start: 4 copper layers, 160 x 100 mm, 110 parts, among them J1 DIN41612_02x16_AC_EvenPins, J10 Conn_01x01, J11 Conn_01x01, J12 Conn_01x01, J2 10Vf, J3 10Vs, J4 ADR, J6 LoSense, J7 GNDf, J8 Conn_01x01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

Commit message: asdf
Routing:
- net /ref/ADR_Pin7: vias 0 -> 1
- net (no net): vias 255 -> 253
Changed lines of the file:
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@@
     )
     (pad_to_mask_clearance 0)
-    (grid_origin 56.195 72.84)
     (pcbplotparams
       (layerselection 0x00010fc_ffffffff)
@@
   (via (at 89.215 70.3) (size 1.5) (drill 0.8) (layers "F.Cu" "B.Cu") (free) (net 0))
   (via (at 76.515 83) (size 1.5) (drill 0.8) (layers "F.Cu" "B.Cu") (free) (net 0))
-  (via (at 81.595 80.46) (size 1.5) (drill 0.8) (layers "F.Cu" "B.Cu") (free) (net 0))
   (via (at 117.155 67.76) (size 1.5) (drill 0.8) (layers "F.Cu" "B.Cu") (free) (net 0))
   (via (at 124.775 70.3) (size 1.5) (drill 0.8) (layers "F.Cu" "B.Cu") (free) (net 0))
@@
   (via (at 76.515 90.62) (size 1.5) (drill 0.8) (layers "F.Cu" "B.Cu") (free) (net 0))
   (via (at 114.615 75.38) (size 1.5) (drill 0.8) (layers "F.Cu" "B.Cu") (free) (net 0))
-  (via (at 89.215 116.02) (size 1.5) (drill 0.8) (layers "F.Cu" "B.Cu") (free) (net 0))
   (via (at 81.595 70.3) (size 1.5) (drill 0.8) (layers "F.Cu" "B.Cu") (free) (net 0))
   (via (at 134.935 70.3) (size 1.5) (drill 0.8) (layers "F.Cu" "B.Cu") (free) (net 0))
@@
   (segment (start 142.394511 141.819511) (end 136.71848 136.14348) (width 0.5) (layer "F.Cu") (net 20))
   (segment (start 123.495 131.26) (end 122.492 131.26) (width 0.5) (layer "F.Cu") (net 20))
+  (via (at 132.715 100) (size 1.5) (drill 0.8) (layers "F.Cu" "B.Cu") (net 20))
   (segment (start 130.109 119.83) (end 130.109 100.715) (width 1) (layer "B.Cu") (net 20))
   (segment (start 131.125 124.91) (end 131.125 101.59) (width 0.5) (layer "B.Cu") (net 20))
@@
   )
   (zone (net 37) (net_name "/DC-DC/rectified+") (layer "F.Cu") (hatch edge 0.508)
-    (priority 1)
+    (priority 2)
     (connect_pads (clearance 0.2))
     (min_thickness 0.1) (filled_areas_thickness no)
@@
   )
   (zone (net 31) (net_name "/DC-DC/12Vf") (layer "F.Cu") (hatch edge 0.508)
-    (priority 1)
+    (priority 2)
     (connect_pads (clearance 0.2))
     (min_thickness 0.1) (filled_areas_thickness no)
@@
       )
     )
-  )
-  (zone (net 0) (net_name "") (layers "In1.Cu" "In2.Cu") (hatch edge 0.508)
-    (connect_pads (clearance 0))
-    (min_thickness 0.127)
-    (keepout (tracks not_allowed) (vias not_allowed) (pads not_allowed ) (copperpour allowed) (footprints allowed))
-    (fill (thermal_gap 0.254) (thermal_bridge_width 0.508))
-    (polygon
-      (pts
-        (xy 128.004948 100)
-        (xy 127.986413 99.183242)
-        (xy 127.930847 98.368165)
-        (xy 127.838363 97.556448)
-        (xy 127.709153 96.749762)
-        (xy 127.543482 95.949768)
-        (xy 127.341692 95.158113)
-        (xy 127.104197 94.376426)
-        (xy 126.831488 93.606318)
-        (xy 126.524124 92.849373)
-        (xy 126.18274 92.10715)
-        (xy 125.808038 91.381178)
-        (xy 125.400789 90.672951)
-        (xy 124.961832 89.983926)
-        (xy 124.492071 89.315524)
-        (xy 123.992473 88.669119)
-        (xy 123.464066 88.046043)
-        (xy 122.907938 87.447579)
-        (xy 122.325235 86.874958)
-        (xy 121.717156 86.32936)
-        (xy 121.084953 85.811907)
-        (xy 120.429927 85.323666)
-        (xy 119.753428 84.865642)
-        (xy 119.056848 84.438777)
-        (xy 118.341621 84.043951)
-        (xy 117.60922 83.681975)
-        (xy 116.861152 83.353597)
-        (xy 116.098959 83.059491)
-        (xy 115.324208 82.800263)
-        (xy 114.538496 82.576447)
-        (xy 113.743439 82.388503)
-        (xy 112.940675 82.23682)
-        (xy 112.131857 82.121708)
-        (xy 111.31865 82.043405)
-        (xy 110.502728 82.002072)
-        (xy 109.68577 81.997794)
-        (xy 108.86946 82.030581)
-        (xy 108.055477 82.100364)
-        (xy 107.245498 82.206999)
-        (xy 106.44119 82.350268)
-        (xy 105.644209 82.529876)
-        (xy 104.856196 82.745452)
-        (xy 104.078773 82.996553)
-        (xy 103.313541 83.282661)
-        (xy 102.562076 83.603188)
-        (xy 101.825925 83.957474)
-        (xy 101.106602 84.344789)
-        (xy 100.40559 84.764336)
-        (xy 99.724332 85.215251)
-        (xy 99.06423 85.696606)
-        (xy 98.426643 86.20741)
-        (xy 97.812883 86.74661)
-        (xy 97.224216 87.313098)
-        (xy 96.661852 87.905706)
-        (xy 96.126949 88.523214)
-        (xy 95.620609 89.164352)
-        (xy 95.143874 89.827798)
-        (xy 94.697726 90.512188)
-        (xy 94.283083 91.216112)
-        (xy 93.900799 91.938121)
-        (xy 93.551662 92.676728)
-        (xy 93.236388 93.430412)
-        (xy 92.955629 94.197623)
-        (xy 92.709962 94.97678)
-        (xy 92.499893 95.766278)
-        (xy 92.325854 96.564494)
-        (xy 92.188203 97.369783)
-        (xy 92.087225 98.180487)
-        (xy 92.023126 98.994937)
-        (xy 91.996039 99.811456)
-        (xy 92.00602 100.628364)
-        (xy 92.053048 101.443977)
-        (xy 92.137026 102.256618)
-        (xy 92.257782 103.064613)
-        (xy 92.415066 103.866298)
-        (xy 92.608556 104.660023)
-        (xy 92.837852 105.444154)
-        (xy 93.102482 106.217076)
-        (xy 93.401902 106.977198)
-        (xy 93.735495 107.722955)
-        (xy 94.102575 108.452811)
-        (xy 94.502385 109.165264)
-        (xy 94.934102 109.858847)
-        (xy 95.396838 110.532133)
-        (xy 95.88964 111.183733)
-        (xy 96.411493 111.812309)
-        (xy 96.961323 112.416564)
-        (xy 97.537998 112.995255)
-        (xy 98.140331 113.547191)
-        (xy 98.76708 114.071235)
-        (xy 99.416957 114.566309)
-        (xy 100.088623 115.031392)
-        (xy 100.780695 115.465528)
-        (xy 101.491748 115.867823)
-        (xy 102.220319 116.237448)
-        (xy 102.964906 116.573642)
-        (xy 103.723978 116.875713)
-        (xy 104.495972 117.14304)
-        (xy 105.279297 117.375072)
-        (xy 106.072342 117.571331)
-        (xy 106.873474 117.731412)
-        (xy 107.681042 117.854988)
-        (xy 108.493385 117.941802)
-        (xy 109.308829 117.991677)
-        (xy 110.125697 118.004509)
-        (xy 110.942306 117.980273)
-        (xy 111.756975 117.919018)
-        (xy 112.568027 117.82087)
-        (xy 113.373791 117.686031)
-        (xy 114.172609 117.514779)
-        (xy 114.962836 117.307467)
-        (xy 115.742846 117.064521)
-        (xy 116.511032 116.786442)
-        (xy 117.265812 116.473801)
-        (xy 118.005633 116.127244)
-        (xy 118.728972 115.747482)
-        (xy 119.434339 115.335299)
-        (xy 120.120282 114.891543)
-        (xy 120.785389 114.417127)
-        (xy 121.42829 113.913028)
-        (xy 122.047662 113.380284)
-        (xy 122.642229 112.819992)
-        (xy 123.210768 112.233305)
-        (xy 123.752108 111.621432)
-        (xy 124.265134 110.985632)
-        (xy 124.74879 110.327214)
-        (xy 125.20208 109.647534)
-        (xy 125.624072 108.94799)
-        (xy 126.013896 108.230024)
-        (xy 126.370749 107.495114)
-        (xy 126.693897 106.744772)
-        (xy 126.982675 105.980544)
-        (xy 127.236488 105.204002)
-        (xy 127.454813 104.416747)
-        (xy 127.637201 103.620398)
-        (xy 127.783277 102.816594)
-        (xy 127.89274 102.006992)
-        (xy 127.965364 101.193258)
-        (xy 128.000999 100.377067)
-      )
-    )

Commit message: flood of prototyping area
Parts:
- added JP20: Jumper_2_Bridged, Jumper:SolderJumper-2_P1.3mm_Bridged_RoundedPad1.0x1.5mm, F.Cu at (134.6, 97.8)
- moved D4 1.02 mm to (75.5, 105.8)
Routing:
- net /ref/ADR: track 227.0 -> 230.2 mm, vias 1 -> 2
- net /DC-DC/GNDf: track 255.6 -> 258.4 mm
- net /ref/ADR_Pin7: track 348.0 -> 350.5 mm, vias 1 -> 3
- net /ref/ADR_Pin4: track 73.5 -> 75.8 mm, vias 1 -> 2
- net /ref/shield_maybe: track 0.00 -> 1.89 mm, vias 0 -> 3
- net /ref/ADR_Pin8: track 123.6 -> 125.3 mm, vias 1 -> 2
- net /ref/U8_Pin2: track 31.0 -> 30.1 mm
- net /ref/U5_Pin7: track 114.5 -> 115.2 mm
- net /ref/ADR_Pin6: track 82.4 -> 83.0 mm, vias 0 -> 1
- net /ref/ADR_Pin1: track 163.2 -> 163.9 mm
- net /ref/RN1_Pin2: track 16.5 -> 16.8 mm, vias 0 -> 1
- net /ref/ADR_Pin5: vias 1 -> 5
- net /ref/RN1_Pin7: vias 0 -> 1
- net /ref/RN1_Pin6: vias 0 -> 1
- net /ref/RN1_Pin5: vias 0 -> 1
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- added copper zone on In1.Cu, net /ref/shield_maybe
- added copper zone on In2.Cu, net /ref/shield_maybe
- removed copper zone on In1.Cu, net (none)
- removed copper zone on In2.Cu, net (none)
