File: ref.kicad_sch (KiCad schematic)
At the start: 1 part, among them U4 ADR1000

Commit message: asdf
Parts:
- added D3, D4: D, Diode_SMD:D_SOD-123, symbol Device:D
- added Q1: Q_NPN_BCE, Package_TO_SOT_SMD:SOT-223-3_TabPin2, symbol Device:Q_NPN_BCE
- added RN1: 322146, Package_DIP:DIP-14_W7.62mm, symbol ADRmu_Library:322146
- added U5: Opamp_Dual, Package_SO:SOIC-8_3.9x4.9mm_P1.27mm, symbol Device:Opamp_Dual
Connections:
- net at U4.1 (HTR+): now also Q1.3 (E)
- net at U4.2 (HTR-): now also D3.2 (A)
- net at U4.3 (VREF): now also D4.1 (K), RN1.1 (R1.1), RN1.2 (R2.1), RN1.5 (R4.3)
- net at U4.4 (IZSET): now also RN1.3 (R3.1)
- net at U4.5 (CQ1): now also RN1.13 (R2.2)
- net at U4.6 (BQ2): now also RN1.11 (R4.2)
- net at U4.7 (GND): now also RN1.12 (R3.2), RN1.4 (R4.1)
- net at U4.8 (CQ2): now also RN1.14 (R1.2)
Other:
- moved on the sheet: U4A

Commit message: asdf
Parts:
- added C? (x2): 100n, Capacitor_SMD:C_0805_2012Metric, symbol Device:C
- added R?: 1k, Resistor_SMD:R_0805_2012Metric, symbol Device:R
- added R?: 10k, Resistor_SMD:R_0805_2012Metric, symbol Device:R
- added R?: 1M, Resistor_SMD:R_0805_2012Metric, symbol Device:R
Connections:
- net 0Vin: now also D3.1 (K)
- net 12Vin: now also Q1.2 (C)
- net at Q1.3 (E), U4.1 (HTR+): now also C?.1
- net ADR_Pin6: now reaches RN1.11 (R4.2), U4.6 (BQ2)
- net ADR_Pin6: now also R?.1
- net at RN1.12 (R3.2), RN1.4 (R4.1), U4.7 (GND): now also C?.1
- net ADR_Pin8: now reaches RN1.14 (R1.2), U4.8 (CQ2)
- net ADR_Pin8: now also U5.5 (+), C?.2
- net at Q1.1 (B): now also R?.1
- net at U5.6 (-): now also R?.2, R?.2
- net at U5.7: now also R?.2
- new net: C?.2, R?.1
Other:
- moved on the sheet: D3, D4, Q1, RN1A, RN1B, RN1C, RN1D, U4A, U4B, U5B

Commit message: asdf
Parts:
- added unit 6 of RN1
- added unit 7 of RN1
- gave numbers to parts that had none: 5
Connections:
- net ADR_Pin6: now also RN1.11 (R5.2), RN1.4 (R4.1); no longer RN1.11 (R4.2)
- net ADR_Pin8: now also RN1.13 (R2.2); no longer RN1.14 (R1.2)
- net at D4.1 (K), RN1.1 (R2.1), RN1.2 (R2.1)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: now also RN1.5 (R5.1); no longer RN1.5 (R4.3)
- net at U4.5 (CQ1): now also RN1.14 (R1.2); no longer RN1.13 (R2.2)
- net at C8.1, RN1.12 (R3.2), U4.7 (GND): now also RN1.11 (R4.2); no longer RN1.4 (R4.1)
- new net: RN1.7 (R7.1), RN1.9 (R6.2)

Commit message: asdf
Parts:
- added C? (x2): 100n, Capacitor_SMD:C_0805_2012Metric, symbol Device:C
Connections:
- net ADR_Pin6: now also RN1.11 (R4.2); no longer RN1.4 (R4.1)
- net ADR_Pin3: now reaches D4.1 (K), RN1.1 (R2.1), RN1.2 (R2.1), RN1.5 (R5.1), U4.3 (VREF)
- net at D4.2 (A): now also U5.1, C?.1
- net ADR_Pin4: now reaches U5.2 (-)
- net ADR_Pin4: now also RN1.3 (R3.1), U4.4 (IZSET), C?.2
- net ADR_Pin5: now reaches U5.3 (+)
- net ADR_Pin5: now also RN1.14 (R1.2), U4.5 (CQ1), C?.2
- net ADR_Pin7: now reaches C8.1, RN1.12 (R3.2), U4.7 (GND)
- net ADR_Pin7: now also RN1.4 (R4.1), C?.1; no longer RN1.11 (R4.2)
Other:
- moved on the sheet: D4, RN1C, RN1D, U5A

Commit message: asdf
Parts:
- gave numbers to parts that had none: 2
Connections:
- net at RN1.9 (R6.2): now also RN1.9 (R7.2); no longer RN1.7 (R7.1)
Other:
- moved on the sheet: C10, C8, C9, D4, RN1A, RN1B, RN1C, RN1D, RN1E, RN1G, U4B, U5A

Commit message: asdf
Parts:
- added C13: 100n, Capacitor_SMD:C_0805_2012Metric, symbol Device:C
Connections:
- net at U5.4 (V-): now also C13.1
- net at U5.8 (V+): now also C13.2
Other:
- moved on the sheet: U5C
Changed lines of the file:
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@@
+    (stroke (width 0) (type default) (color 0 0 0 0))
+  )
+  (wire (pts (xy 93.98 116.84) (xy 93.98 111.76))
     (stroke (width 0) (type default) (color 0 0 0 0))
   )
@@
     (stroke (width 0) (type default) (color 0 0 0 0))
   )
+  (wire (pts (xy 93.98 111.76) (xy 101.6 111.76))
+    (stroke (width 0) (type default) (color 0 0 0 0))
+  )
   (wire (pts (xy 107.95 44.45) (xy 123.19 44.45))
     (stroke (width 0) (type default) (color 0 0 0 0))
@@
     (stroke (width 0) (type default) (color 0 0 0 0))
   )
+  (wire (pts (xy 101.6 111.76) (xy 101.6 113.03))
+    (stroke (width 0) (type default) (color 0 0 0 0))
+  )
   (wire (pts (xy 179.07 85.09) (xy 179.07 59.69))
     (stroke (width 0) (type default) (color 0 0 0 0))
@@
     (stroke (width 0) (type default) (color 0 0 0 0))
   )
+  (wire (pts (xy 101.6 128.27) (xy 101.6 129.54))
+    (stroke (width 0) (type default) (color 0 0 0 0))
+  )
   (wire (pts (xy 93.98 97.79) (xy 107.95 97.79))
     (stroke (width 0) (type default) (color 0 0 0 0))
@@
     (stroke (width 0) (type default) (color 0 0 0 0))
   )
+  (wire (pts (xy 93.98 129.54) (xy 101.6 129.54))
+    (stroke (width 0) (type default) (color 0 0 0 0))
+  )
   (wire (pts (xy 125.73 82.55) (xy 125.73 97.79))
     (stroke (width 0) (type default) (color 0 0 0 0))
@@
   )
   (wire (pts (xy 148.59 74.93) (xy 148.59 97.79))
+    (stroke (width 0) (type default) (color 0 0 0 0))
+  )
+  (wire (pts (xy 93.98 124.46) (xy 93.98 129.54))
     (stroke (width 0) (type default) (color 0 0 0 0))
   )
@@
     (pin "2")
   )
-  (symbol (lib_id "Device:Opamp_Dual") (at 248.92 118.11 0) (unit 3)
-    (in_bom yes) (on_board yes) (fields_autoplaced)
-    (property "Reference" "U5" (id 0) (at 247.65 116.8399 0)
-      (effects (font (size 1.27 1.27)) (justify left))
-    )
-    (property "Value" "Opamp_Dual" (id 1) (at 247.65 119.3799 0)
-      (effects (font (size 1.27 1.27)) (justify left))
-    )
-    (property "Footprint" "" (id 2) (at 248.92 118.11 0)
-      (effects (font (size 1.27 1.27)) hide)
-    )
-    (property "Datasheet" "~" (id 3) (at 248.92 118.11 0)
+  (symbol (lib_id "Device:Opamp_Dual") (at 104.14 120.65 0) (unit 3)
+    (in_bom yes) (on_board yes) (fields_autoplaced)
+    (property "Reference" "U5" (id 0) (at 102.87 119.3799 0)
+      (effects (font (size 1.27 1.27)) (justify left))
+    )
+    (property "Value" "Opamp_Dual" (id 1) (at 102.87 121.9199 0)
+      (effects (font (size 1.27 1.27)) (justify left))
+    )
+    (property "Footprint" "" (id 2) (at 104.14 120.65 0)
+      (effects (font (size 1.27 1.27)) hide)
+    )
+    (property "Datasheet" "~" (id 3) (at 104.14 120.65 0)
       (effects (font (size 1.27 1.27)) hide)
     )
@@
     (pin "14")
   )
+  (symbol (lib_id "Device:C") (at 93.98 120.65 180) (unit 1)
+    (in_bom yes) (on_board yes) (fields_autoplaced)
+    (property "Reference" "C13" (id 0) (at 90.17 119.3799 0)
+      (effects (font (size 1.27 1.27)) (justify left))
+    )
+    (property "Value" "100n" (id 1) (at 90.17 121.9199 0)
+      (effects (font (size 1.27 1.27)) (justify left))
+    )
+    (property "Footprint" "Capacitor_SMD:C_0805_2012Metric" (id 2) (at 93.0148 116.84 0)
+      (effects (font (size 1.27 1.27)) hide)
+    )
+    (property "Datasheet" "~" (id 3) (at 93.98 120.65 0)
+      (effects (font (size 1.27 1.27)) hide)
+    )
+    (pin "1")
+    (pin "2")
+  )
   (symbol (lib_id "ADRmu_Library:322146") (at 123.19 50.8 0) (unit 2)

Commit message: added i2c temperature sensor and eeprom
Connections:
- net ADR_Pin3 renamed ADR
Changed lines of the file:
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@@
+    (stroke (width 0) (type default) (color 0 0 0 0))
+  )
+  (wire (pts (xy 132.08 33.02) (xy 209.55 33.02))
     (stroke (width 0) (type default) (color 0 0 0 0))
   )
@@
   )
   (wire (pts (xy 49.53 82.55) (xy 49.53 85.09))
+    (stroke (width 0) (type default) (color 0 0 0 0))
+  )
+  (wire (pts (xy 132.08 44.45) (xy 132.08 33.02))
     (stroke (width 0) (type default) (color 0 0 0 0))
   )
@@
     (effects (font (size 1.27 1.27)) (justify right))
   )
-  (hierarchical_label "ADRforce" (shape output) (at 217.17 71.12 0)
+  (hierarchical_label "ADR" (shape output) (at 209.55 33.02 0)
     (effects (font (size 1.27 1.27)) (justify left))
   )
@@
     (effects (font (size 1.27 1.27)) (justify left))
   )
-  (hierarchical_label "ADRsense" (shape output) (at 217.17 77.47 0)
-    (effects (font (size 1.27 1.27)) (justify left))
-  )

Commit message: asas
Parts:
- added R13: dnp, Resistor_SMD:R_0805_2012Metric, symbol Device:R
- added R14: dnp, Crystal:Crystal_HC52-U_Vertical, symbol Device:R
- added R15, R17: 0, Resistor_SMD:R_0805_2012Metric, symbol Device:R
- added R16, R18: 0, Crystal:Crystal_HC52-U_Vertical, symbol Device:R
Connections:
- net ADR_Pin7: now also R15.1, R16.1, R17.1, R18.1; no longer RN1.12 (R3.2), RN1.4 (R4.1)
- new net: R17.2, R18.2, RN1.12 (R3.2)
- new net: R15.2, R16.2, RN1.4 (R4.1)
- new net: R13.1, R14.1
- new net: R13.2, R14.2
Other:
- moved on the sheet: C13, U5C
