File: ADRmu.kicad_sch (KiCad schematic)
At the start: 6 parts, among them J1 DIN41612_02x16_AC_EvenPins, J2 10Vf, J3 10Vs, J4 ADR, J6 return, J7 guard

Commit message: started proto area
Parts:
- added NT1: NetTie_2, NetTie:NetTie-2_SMD_Pad0.5mm, symbol Device:NetTie_2
- J6: value return -> LoSense
- J7: value guard -> GND
Connections:
- net ref/guard renamed ref/GND
- net ref/return: no longer names the net of J1.a28 (Pin_a28), J1.c28 (Pin_c28)
- net ref/return: now also NT1.1; no longer J6.1 (Pin_1)
- new net ref/LoSense: J6.1 (Pin_1), NT1.2
Other:
- sheet ref ports: added GND, LoSense; removed guard, return
Changed lines of the file:
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@@
   (junction (at 68.58 74.93) (diameter 0) (color 0 0 0 0)
   )
+  (junction (at 68.58 110.49) (diameter 0) (color 0 0 0 0)
+  )
   (junction (at 228.6 55.88) (diameter 0) (color 0 0 0 0)
   )
+  (junction (at 68.58 107.95) (diameter 0) (color 0 0 0 0)
+  )
   (junction (at 68.58 97.79) (diameter 0) (color 0 0 0 0)
   )
@@
   (junction (at 68.58 77.47) (diameter 0) (color 0 0 0 0)
   )
-  (junction (at 68.58 107.95) (diameter 0) (color 0 0 0 0)
+  (junction (at 228.6 116.84) (diameter 0) (color 0 0 0 0)
   )
   (junction (at 55.88 77.47) (diameter 0) (color 0 0 0 0)
@@
   (junction (at 52.07 92.71) (diameter 0) (color 0 0 0 0)
   )
-  (junction (at 68.58 110.49) (diameter 0) (color 0 0 0 0)
-  )
-  (junction (at 228.6 116.84) (diameter 0) (color 0 0 0 0)
-  )
   (junction (at 68.58 95.25) (diameter 0) (color 0 0 0 0)
   )
@@
     (stroke (width 0) (type default) (color 0 0 0 0))
   )
-  (wire (pts (xy 68.58 107.95) (xy 77.47 107.95))
+  (wire (pts (xy 228.6 116.84) (xy 231.14 116.84))
     (stroke (width 0) (type default) (color 0 0 0 0))
   )
@@
     (stroke (width 0) (type default) (color 0 0 0 0))
   )
-  (wire (pts (xy 228.6 116.84) (xy 215.9 116.84))
-    (stroke (width 0) (type default) (color 0 0 0 0))
-  )
   (wire (pts (xy 55.88 97.79) (xy 68.58 97.79))
     (stroke (width 0) (type default) (color 0 0 0 0))
@@
     (stroke (width 0) (type default) (color 0 0 0 0))
   )
+  (wire (pts (xy 68.58 107.95) (xy 69.85 107.95))
+    (stroke (width 0) (type default) (color 0 0 0 0))
+  )
+  (wire (pts (xy 215.9 116.84) (xy 228.6 116.84))
+    (stroke (width 0) (type default) (color 0 0 0 0))
+  )
   (wire (pts (xy 68.58 97.79) (xy 83.82 97.79))
     (stroke (width 0) (type default) (color 0 0 0 0))
@@
     (stroke (width 0) (type default) (color 0 0 0 0))
   )
-  (wire (pts (xy 231.14 116.84) (xy 228.6 116.84))
-    (stroke (width 0) (type default) (color 0 0 0 0))
-  )
   (wire (pts (xy 77.47 153.67) (xy 242.57 153.67))
     (stroke (width 0) (type default) (color 0 0 0 0))
@@
     (stroke (width 0) (type default) (color 0 0 0 0))
   )
-  (wire (pts (xy 74.93 156.21) (xy 74.93 110.49))
-    (stroke (width 0) (type default) (color 0 0 0 0))
-  )
   (wire (pts (xy 55.88 110.49) (xy 68.58 110.49))
     (stroke (width 0) (type default) (color 0 0 0 0))
@@
     (stroke (width 0) (type default) (color 0 0 0 0))
   )
-  (wire (pts (xy 74.93 110.49) (xy 68.58 110.49))
-    (stroke (width 0) (type default) (color 0 0 0 0))
-  )
   (wire (pts (xy 72.39 113.03) (xy 68.58 113.03))
     (stroke (width 0) (type default) (color 0 0 0 0))
@@
     (stroke (width 0) (type default) (color 0 0 0 0))
   )
+  (wire (pts (xy 74.93 110.49) (xy 74.93 156.21))
+    (stroke (width 0) (type default) (color 0 0 0 0))
+  )
+  (wire (pts (xy 74.93 107.95) (xy 77.47 107.95))
+    (stroke (width 0) (type default) (color 0 0 0 0))
+  )
+  (wire (pts (xy 68.58 110.49) (xy 74.93 110.49))
+    (stroke (width 0) (type default) (color 0 0 0 0))
+  )
   (wire (pts (xy 80.01 105.41) (xy 80.01 151.13))
     (stroke (width 0) (type default) (color 0 0 0 0))
@@
   (wire (pts (xy 77.47 107.95) (xy 77.47 153.67))
     (stroke (width 0) (type default) (color 0 0 0 0))
+  )
+  (symbol (lib_id "Device:NetTie_2") (at 72.39 107.95 0) (unit 1)
+    (in_bom yes) (on_board yes) (fields_autoplaced)
+    (property "Reference" "NT1" (id 0) (at 72.39 102.87 0))
+    (property "Value" "NetTie_2" (id 1) (at 72.39 105.41 0))
+    (property "Footprint" "NetTie:NetTie-2_SMD_Pad0.5mm" (id 2) (at 72.39 107.95 0)
+      (effects (font (size 1.27 1.27)) hide)
+    )
+    (property "Datasheet" "~" (id 3) (at 72.39 107.95 0)
+      (effects (font (size 1.27 1.27)) hide)
+    )
+    (pin "1")
+    (pin "2")
   )
   (symbol (lib_id "Connector_Generic:Conn_01x01") (at 236.22 86.36 0) (mirror x) (unit 1)
@@
     (in_bom yes) (on_board yes) (fields_autoplaced)
     (property "Reference" "J6" (id 0) (at 236.22 110.49 0))
-    (property "Value" "return" (id 1) (at 236.22 113.03 0))
+    (property "Value" "LoSense" (id 1) (at 236.22 113.03 0))
     (property "Footprint" "Connector_Wire:SolderWire-1sqmm_1x01_D1.4mm_OD3.9mm" (id 2) (at 236.22 116.84 0)
       (effects (font (size 1.27 1.27)) hide)
@@
     (in_bom yes) (on_board yes) (fields_autoplaced)
     (property "Reference" "J7" (id 0) (at 236.22 125.73 0))
-    (property "Value" "guard" (id 1) (at 236.22 128.27 0))
+    (property "Value" "GND" (id 1) (at 236.22 128.27 0))
     (property "Footprint" "Connector_Wire:SolderWire-1sqmm_1x01_D1.4mm_OD3.9mm" (id 2) (at 236.22 132.08 0)
       (effects (font (size 1.27 1.27)) hide)
@@
       (effects (font (size 1.27 1.27)) (justify right))
     )
-    (pin "guard" output (at 215.9 132.08 0)
+    (pin "12Vin" input (at 157.48 76.2 180)
+      (effects (font (size 1.27 1.27)) (justify left))
+    )
+    (pin "0Vin" input (at 157.48 111.76 180)
+      (effects (font (size 1.27 1.27)) (justify left))
+    )
+    (pin "ADR" output (at 215.9 86.36 0)
       (effects (font (size 1.27 1.27)) (justify right))
     )
-    (pin "return" output (at 215.9 116.84 0)
+    (pin "GND" output (at 215.9 132.08 0)
       (effects (font (size 1.27 1.27)) (justify right))
     )
-    (pin "12Vin" input (at 157.48 76.2 180)
-      (effects (font (size 1.27 1.27)) (justify left))
-    )
-    (pin "0Vin" input (at 157.48 111.76 180)
-      (effects (font (size 1.27 1.27)) (justify left))
-    )
-    (pin "ADR" output (at 215.9 86.36 0)
+    (pin "LoSense" output (at 215.9 116.84 0)
       (effects (font (size 1.27 1.27)) (justify right))
     )
@@
     )
     (path "/30570277-0b2d-44ac-9416-b1ae1209d471"
-      (reference "J6") (unit 1) (value "return") (footprint "Connector_Wire:SolderWire-1sqmm_1x01_D1.4mm_OD3.9mm")
+      (reference "J6") (unit 1) (value "LoSense") (footprint "Connector_Wire:SolderWire-1sqmm_1x01_D1.4mm_OD3.9mm")
     )
     (path "/e45d5717-29b8-4b31-b3f8-99a046e18c84"
-      (reference "J7") (unit 1) (value "guard") (footprint "Connector_Wire:SolderWire-1sqmm_1x01_D1.4mm_OD3.9mm")
+      (reference "J7") (unit 1) (value "GND") (footprint "Connector_Wire:SolderWire-1sqmm_1x01_D1.4mm_OD3.9mm")
     )
     (path "/b2eac6f7-6f2b-41aa-9eec-9c2e749d1013/00d886bb-f578-4690-8703-0d82aa33913b"
@@
       (reference "JP4") (unit 1) (value "Jumper_2_Open") (footprint "Jumper:SolderJumper-2_P1.3mm_Open_RoundedPad1.0x1.5mm")
     )
+    (path "/1705e2a0-ea24-49d8-be00-c4975f9b9685"
+      (reference "NT1") (unit 1) (value "NetTie_2") (footprint "NetTie:NetTie-2_SMD_Pad0.5mm")
+    )
     (path "/027929a1-62dd-40f4-83d4-39d0de3b1543/89dd6cef-9682-496d-9d3c-46b557a5d343"
       (reference "Q1") (unit 1) (value "Q_NPN_BCE") (footprint "Package_TO_SOT_SMD:SOT-223-3_TabPin2")
@@
       (reference "R22") (unit 1) (value "49.9k") (footprint "Resistor_SMD:R_0805_2012Metric")
     )
+    (path "/027929a1-62dd-40f4-83d4-39d0de3b1543/49148cb7-730f-439c-bfcf-650a4b0abde3"
+      (reference "R23") (unit 1) (value "dnp") (footprint "Resistor_SMD:R_0805_2012Metric")
+    )
+    (path "/027929a1-62dd-40f4-83d4-39d0de3b1543/b2c4815f-a979-4a2a-8bcd-21b3f043d2fa"
+      (reference "R24") (unit 1) (value "dnp") (footprint "Crystal:Crystal_HC52-U_Vertical")
+    )
+    (path "/027929a1-62dd-40f4-83d4-39d0de3b1543/04c2e7e5-0afd-4525-970b-5a890e945752"
+      (reference "R25") (unit 1) (value "dnp") (footprint "Resistor_SMD:R_0805_2012Metric")
+    )
+    (path "/027929a1-62dd-40f4-83d4-39d0de3b1543/0b89163e-f67a-456d-a72a-b7bda61551c9"
+      (reference "R26") (unit 1) (value "dnp") (footprint "Crystal:Crystal_HC52-U_Vertical")
+    )
+    (path "/027929a1-62dd-40f4-83d4-39d0de3b1543/933f9b00-a846-4a32-9364-42d908a93e19"
+      (reference "R27") (unit 1) (value "dnp") (footprint "Resistor_SMD:R_0805_2012Metric")
+    )
+    (path "/027929a1-62dd-40f4-83d4-39d0de3b1543/ae87217e-11f9-4fc6-9d00-6532f0c2c91f"
+      (reference "R28") (unit 1) (value "dnp") (footprint "Crystal:Crystal_HC52-U_Vertical")
+    )
+    (path "/027929a1-62dd-40f4-83d4-39d0de3b1543/73810e81-4de6-4455-9d03-fee69b696ce2"
+      (reference "R29") (unit 1) (value "dnp") (footprint "Resistor_SMD:R_0805_2012Metric")
+    )
+    (path "/027929a1-62dd-40f4-83d4-39d0de3b1543/17e0a92d-9678-4bb5-9350-2724578c034e"
+      (reference "R30") (unit 1) (value "dnp") (footprint "Crystal:Crystal_HC52-U_Vertical")
+    )
+    (path "/027929a1-62dd-40f4-83d4-39d0de3b1543/4d665021-6b9d-4792-8432-4ee92e12013e"
+      (reference "R31") (unit 1) (value "dnp") (footprint "Resistor_SMD:R_0805_2012Metric")
+    )
+    (path "/027929a1-62dd-40f4-83d4-39d0de3b1543/c2bd0489-b14f-44da-9320-e8d1549c7ac2"
+      (reference "R32") (unit 1) (value "dnp") (footprint "Crystal:Crystal_HC52-U_Vertical")
+    )
     (path "/027929a1-62dd-40f4-83d4-39d0de3b1543/61e33ddb-fb2f-4483-96fd-ca725420cb1a"

Commit message: the small reset
Parts:
- removed NT1: NetTie_2, NetTie:NetTie-2_SMD_Pad0.5mm, symbol Device:NetTie_2
- J7: value GND -> GNDf
Connections:
- net ref/LoSense: now also J1.a28 (Pin_a28), J1.c28 (Pin_c28)
- net DC-DC/Vin+ renamed DC-DC/Ext_Vin+
- net DC-DC/Vin- renamed DC-DC/Ext_GND
- net ref/GND renamed DC-DC/GNDf
Other:
- sheet DC-DC ports: added 12Vf, Ext_GND, Ext_Vin+, GNDf; removed 0Vout, 12Vout, Vin+, Vin-
- sheet ref ports: added DC_DC_GND, DC_DC_Vin+; removed 0Vin, 12Vin, GND
