File: ADRmu.kicad_sch (KiCad schematic)
At the start: 6 parts, among them J1 DIN41612_02x16_AC_EvenPins, J2 10Vf, J3 10Vs, J4 ADR, J6 LoSense, J7 GNDf

Commit message: added dubious flightless birb
Parts:
- added SYM101: SYM_Earth_Protective_Large, ADRmu_Library:osmu_logo, symbol Graphic:SYM_Earth_Protective_Large
Changed lines of the file:
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@@
     (pin "1")
+  )
+  (symbol (lib_id "Graphic:SYM_Earth_Protective_Large") (at 146.05 177.8 0) (unit 1)
+    (in_bom yes) (on_board yes) (fields_autoplaced)
+    (property "Reference" "SYM101" (id 0) (at 146.05 172.72 0)
+      (effects (font (size 1.27 1.27)) hide)
+    )
+    (property "Value" "SYM_Earth_Protective_Large" (id 1) (at 146.05 182.245 0)
+      (effects (font (size 1.27 1.27)) hide)
+    )
+    (property "Footprint" "ADRmu_Library:osmu_logo" (id 2) (at 146.05 176.53 0)
+      (effects (font (size 1.27 1.27)) hide)
+    )
+    (property "Datasheet" "~" (id 3) (at 146.05 176.53 0)
+      (effects (font (size 1.27 1.27)) hide)
+    )
   )
   (symbol (lib_id "Connector:DIN41612_02x16_AC_EvenPins") (at 60.96 92.71 0) (unit 1)
@@
       (reference "RN201") (unit 7) (value "322146") (footprint "Package_DIP:DIP-14_W7.62mm")
     )
+    (path "/b6049450-f12f-4eca-adfb-237ec3a8e84f"
+      (reference "SYM101") (unit 1) (value "SYM_Earth_Protective_Large") (footprint "ADRmu_Library:osmu_logo")
+    )
     (path "/b2eac6f7-6f2b-41aa-9eec-9c2e749d1013/a8cc43c4-7914-481f-bd3d-67efa0fecedb"
