File: module_reference/ADRmu.kicad_pcb (KiCad board)
At the start: 4 copper layers, 160 x 100 mm, 145 parts, among them J101 Harting 09042326831, J102 10Vf, J103 10Vs, J104 7Vref, J105 Lo, J301 Conn_01x01, J302 Conn_01x01, J303 Conn_01x01, J304 Conn_01x01, J305 Conn_01x01, Q201 BDP949, Q301 MMBT3904, U201 ADR1000, U202 OPA2140, U203 ADA4523-1, U301 L78L33_SOT89, U302 LT3439, U303 24LC02, U304 TMP117, U305 LT3045xMSE

Commit message: rev 0.4 layout step
Parts:
- removed FL301: B82793C0206N265, ADRmu_Library:Filter_EPCOS_B82793C0
- removed the JP203 at (75.9, 120.1)
- removed JP305, JP306: Jumper_2_Open, Jumper:SolderJumper-2_P1.3mm_Open_RoundedPad1.0x1.5mm
- removed the R203 at (75.9, 118.2)
- removed the R205 at (75.9, 120.1)
- NT201: footprint NetTie:NetTie-2_SMD_Pad0.5mm -> NetTie:NetTie-2_SMD_Pad2.0mm
- Q201: value BDP949 -> BD135; footprint Package_TO_SOT_SMD:SOT-223-3_TabPin2 -> Package_TO_SOT_THT:TO-126-3_Vertical
- SYM101: moved to B.Cu
- moved R203 71.0 mm to (87.0, 132.8), turned to 90 degrees
- moved R308 56.7 mm to (160.0, 114.0)
- moved Q301 53.8 mm to (161.1, 118.0)
- moved JP224 40.5 mm to (80.0, 113.8), turned to 90 degrees
- moved JP221 40.4 mm to (83.0, 113.8), turned to -90 degrees
- moved JP227 40.3 mm to (86.0, 113.8), turned to 90 degrees
- moved RN204 34.4 mm to (87.3, 109.8), turned to 180 degrees
- moved C308 31.7 mm to (164.0, 71.0)
- moved U303 31.7 mm to (161.3, 70.9)
- moved RN201 31.3 mm to (91.6, 91.1), turned to 0 degrees
- moved D304 23.0 mm to (200.0, 130.5)
- moved NT201 22.4 mm to (150.0, 87.3)
- moved Q201 21.0 mm to (93.0, 70.8), turned to -135 degrees
- moved J304 20.0 mm to (185.0, 130.0)
- moved D303 19.4 mm to (189.0, 130.5)
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- renumbered C303 to C302, C302 to C303, C308 to C307, C309 to C308, C310 to C309, C311 to C310, C307 to C311, JP204 to JP202, JP205 to JP203, JP206 to JP204, JP207 to JP205, JP208 to JP206, JP209 to JP207, JP210 to JP208, JP211 to JP209, JP212 to JP210, JP213 to JP211, JP214 to JP212, JP215 to JP213, JP216 to JP214, JP217 to JP215, JP218 to JP216, JP219 to JP217, JP220 to JP218, JP221 to JP219, JP222 to JP220, JP223 to JP221, JP224 to JP222, JP225 to JP223, JP226 to JP224, JP227 to JP225, JP228 to JP226, JP229 to JP227, R204 to R203, R206 to R204, R207 to R205, R208 to R206, R209 to R207, R210 to R208, R211 to R209, R212 to R210, R213 to R211, R214 to R212, R215 to R213, R216 to R214, R217 to R215, R218 to R216, R219 to R217, R220 to R218, R221 to R219, R222 to R220, R223 to R221, R224 to R222, R225 to R223, R226 to R224, R227 to R225, R228 to R226, R229 to R227, R303 to R302, R302 to R303, U304 to U303, U303 to U304
Connections:
- C307 pad 1: /DC-DC/rectified+ -> /DC-DC/filtered+
- C307 pad 2: /DC-DC/rectified- -> GNDA
- D302 pad 1: /DC-DC/rectified+ -> /DC-DC/filtered+
- D303 pad 2: /DC-DC/rectified- -> GNDA
- D304 pad 1: /DC-DC/rectified+ -> /DC-DC/filtered+
- D305 pad 2: /DC-DC/rectified- -> GNDA
- J101 pad a14: /DC-DC/status -> unconnected-(J101-Pada14)
- J101 pad a24: unconnected-(J101-Pada24) -> Earth
- J101 pad c14: /DC-DC/status -> unconnected-(J101-Padc14)
- J101 pad c24: unconnected-(J101-Padc24) -> Earth
- JP201 pad 2: /ref/RN201_Pin3 -> /ref/RN201_Pin15
- Q201 pad 1: /ref/Q201_base -> /ref/heater+
- Q201 pad 3: /ref/heater+ -> /ref/Q201_base
- R201 pad 2: /ref/RN201_Pin3 -> /ref/RN201_Pin15
- R202 pad 2: /ref/RN201_Pin3 -> /ref/RN201_Pin15
- RN201 pad 1: /ref/RN201_Pin8 -> /ref/7Vref
- RN201 pad 11: /ref/RN201_Pin14 -> /ref/ADR_Pin7
- RN201 pad 12: /ref/ADR_Pin6 -> /ref/RN201_Pin10
- RN201 pad 13: /ref/RN201_Pin14 -> /ref/ADR_Pin7
- RN201 pad 15: /ref/RN201_Pin16 -> /ref/RN201_Pin15
- RN201 pad 16: /ref/RN201_Pin16 -> /ref/RN201_Pin14
- RN201 pad 2: /ref/RN201_Pin2 -> /ref/ADR_Pin6
- RN201 pad 3: /ref/RN201_Pin3 -> /ref/RN201_Pin5
- RN201 pad 4: /ref/7Vref -> /ref/ADR_Pin6
- RN201 pad 5: /ref/ADR_Pin7 -> /ref/RN201_Pin5
- RN201 pad 6: /ref/RN201_Pin7 -> /ref/ADR_Pin6
- RN201 pad 7: /ref/RN201_Pin7 -> /ref/ADR_Pin6
- RN201 pad 8: /ref/RN201_Pin8 -> /ref/ADR_Pin6
- RN201 pad 9: /ref/RN201_Pin10 -> /ref/ADR_Pin7
Routing:
- net GNDA: track 174.4 -> 356.1 mm, vias 17 -> 11
- net /DC-DC/status_LED: track 259.9 -> 131.6 mm
- net /ref/U202B_out: track 115.1 -> 6.08 mm
- net /ref/Q201_base: track 3.04 -> 74.3 mm, vias 0 -> 1
- net /ref/10Vsense: track 161.8 -> 96.1 mm
- net /ref/ADR_Pin8: track 118.6 -> 69.7 mm
- net /DC-DC/PG: track 57.9 -> 11.2 mm, vias 2 -> 0
- net /DC-DC/12Vf: track 185.9 -> 139.6 mm, vias 29 -> 2
- net /DC-DC/SCL: track 169.5 -> 125.7 mm, vias 2 -> 1
- net /DC-DC/SDA: track 161.3 -> 118.0 mm
- net /ref/ADR_Pin6: track 139.9 -> 98.6 mm
- net GND: track 222.3 -> 182.2 mm, vias 17 -> 13
- net /DC-DC/status: track 39.2 -> 3.02 mm
- net /ref/U203_-in: track 78.6 -> 42.9 mm
- net /ref/heater+: track 164.7 -> 129.6 mm, vias 2 -> 1
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- added copper zone on B.Cu, net /ref/ADR_Pin3
- added copper zone on B.Cu, net Earth
- added copper zone on F.Cu, net Earth
- removed copper zone on In1.Cu, net +12V
- removed copper zone on In2.Cu, net +12V
- removed copper zone on B.Cu, net /DC-DC/12Vf
- removed copper zone on B.Cu, net /ref/ADR_Pin4
- removed copper zone on F.Cu, net /ref/ADR_Pin4
- removed copper zone on B.Cu, net /ref/ADR_Pin7
- removed copper zone on F.Cu, net /ref/ADR_Pin7
- removed copper zone on F.Cu, net /ref/ADR_Pin8
- removed copper zone on B.Cu, net /ref/heater+
- removed copper zone on F.Cu, net /ref/heater-
Other:
- board text added: "ADRmu 10V Standard Rev 0.4"
- board text removed: "ADRmu 10V Standard Rev 0.3"

Commit message: rev 0.4 layout done
Parts:
- SYM101: moved to F.Cu
- moved SYM101 139.7 mm to (76.5, 59.0), turned to 0 degrees
- moved C201 7.29 mm to (92.0, 133.0), turned to 90 degrees
- moved R204 7.01 mm to (90.0, 132.5)
- moved C203 3.79 mm to (94.0, 133.0), turned to 90 degrees
- moved C209 2.56 mm to (145.1, 132.8), turned to 90 degrees
- moved R205 2.20 mm to (96.0, 128.0), turned to 180 degrees
- moved C307 1.99 mm to (176.7, 128.0)
- moved R227 0.28 mm to (143.7, 127.5)
- moved C206 0.16 mm to (132.7, 128.0)
Routing:
- net +12V: track 58.9 -> 15.1 mm
- net +3V3: track 61.7 -> 42.6 mm, vias 6 -> 5
- net /DC-DC/SDA: track 118.0 -> 129.0 mm
- net /DC-DC/SCL: track 125.7 -> 136.4 mm
- net /ref/ADR_Pin6: track 98.6 -> 91.2 mm
- net /DC-DC/status_LED: track 131.6 -> 124.6 mm
- net /ref/ADR_Pin8: track 69.7 -> 64.4 mm
- net GND: track 182.2 -> 177.8 mm, vias 13 -> 11
- net /ref/10Vforce: track 97.1 -> 93.1 mm
- net /DC-DC/pwr_LED: track 155.9 -> 158.8 mm
- net /DC-DC/xformer_B: track 9.25 -> 6.70 mm
- net /ref/U202B_-in: track 4.61 -> 6.85 mm
- net /DC-DC/xformer_A: track 9.16 -> 7.18 mm
- net /ref/heater+: track 129.6 -> 130.7 mm
- net /DC-DC/filtered+: track 51.9 -> 51.2 mm
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- added copper zone on B.Cu, net +12V
- added copper zone on B.Cu, net +3V3
- removed copper zone on B.Cu, net GND

Commit message: asdf
Changed lines of the file:
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@@
     (property "Sheetfile" "dcdc.kicad_sch")
     (property "Sheetname" "DC-DC")
-    (attr exclude_from_pos_files)
+    (property "exclude_from_bom" "")
+    (attr exclude_from_pos_files exclude_from_bom)
     (fp_text reference "JP309" (at 0.75236 -6.5029 90) (layer "F.SilkS")
       (effects (font (size 1 1) (thickness 0.15)))
@@
     (property "Sheetname" "DC-DC")
     (attr smd)
-    (fp_text reference "R301" (at 3.712 0.279 90) (layer "F.SilkS")
+    (fp_text reference "R301" (at 2.412 2.604 180) (layer "F.SilkS")
       (effects (font (size 1 1) (thickness 0.15)))
     )
@@
     (property "Sheetname" "DC-DC")
     (attr smd)
-    (fp_text reference "U301" (at 3.302 0) (layer "F.SilkS")
+    (fp_text reference "U301" (at 1.9316 4.4406) (layer "F.SilkS")
       (effects (font (size 1 1) (thickness 0.15)))
     )
@@
     (property "Sheetfile" "dcdc.kicad_sch")
     (property "Sheetname" "DC-DC")
-    (attr exclude_from_pos_files)
+    (property "exclude_from_bom" "")
+    (attr exclude_from_pos_files exclude_from_bom)
     (fp_text reference "JP308" (at 0.75236 -5.9629 90) (layer "F.SilkS")
       (effects (font (size 1 1) (thickness 0.15)))
@@
     (property "Sheetfile" "dcdc.kicad_sch")
     (property "Sheetname" "DC-DC")
-    (attr exclude_from_pos_files)
+    (property "exclude_from_bom" "")
+    (attr exclude_from_pos_files exclude_from_bom)
     (fp_text reference "JP307" (at 0.75236 -7.0429 90) (layer "F.SilkS")
       (effects (font (size 1 1) (thickness 0.15)))
@@
     (property "Sheetname" "DC-DC")
     (attr smd)
-    (fp_text reference "C301" (at 3.944 0 90) (layer "F.SilkS")
+    (fp_text reference "C301" (at 2.444 -0.5 180) (layer "F.SilkS")
       (effects (font (size 1 1) (thickness 0.15)))
     )
@@
     (property "Sheetname" "DC-DC")
     (attr smd)
-    (fp_text reference "R302" (at 3.712 -0.157 90) (layer "F.SilkS")
+    (fp_text reference "R302" (at 2.412 -2.332 180) (layer "F.SilkS")
       (effects (font (size 1 1) (thickness 0.15)))
     )
@@
     (property "Sheetname" "DC-DC")
     (attr smd)
-    (fp_text reference "C304" (at 3.812 0.111 90) (layer "F.SilkS")
+    (fp_text reference "C304" (at 2.412 0.111 180) (layer "F.SilkS")
       (effects (font (size 1 1) (thickness 0.15)))
     )

Commit message: asdf
Parts:
- C303: value 1000u 25V -> 470u 25V
- R303, R308: value 10k -> 49k9
- U304: value 24LC02 -> BR24H64FVM
- renumbered JP204 to JP205, JP205 to JP206, JP206 to JP207, JP207 to JP208, JP208 to JP209, JP209 to JP210, JP210 to JP211, JP211 to JP212, JP212 to JP213, JP213 to JP214, JP214 to JP215, JP215 to JP216, JP216 to JP217, JP217 to JP218, JP218 to JP219, JP219 to JP220, JP220 to JP221, JP221 to JP222, JP222 to JP223, JP223 to JP224, JP224 to JP225, JP225 to JP226, JP226 to JP227, JP227 to JP228, JP307 to JP305, JP308 to JP306, JP309 to JP307
