File: module_reference/ADRmu.kicad_sch (KiCad schematic)
At the start: 7 parts, among them J101 Harting 09042326831, J102 10Vf, J103 10Vs, J104 7Vref, J105 Lo

Commit message: Reference board Rev 0.5 schematic
Connections:
- net DC-DC/Ext_GND renamed DC-DC/GND
- net DC-DC/Ext_Vin+ renamed DC-DC/+12V
- net ref/Lo renamed ref/ADR_Pin7
Other:
- sheet DC-DC ports: added +12V, GND; removed Ext_GND, Ext_Vin+, status
- sheet ref ports: added ADR_Pin7; removed Lo
