File: module_reference/adrmu6layer.kicad_pcb (KiCad board)
At the start: 6 copper layers, 160 x 100 mm, 218 parts, among them J101 Harting 09042326831, J102 OutHf, J103 OutHs, J104 7Vref, J105 Lo, J106 12VinC, J107 OutLs, J108 OutLf, J201 Conn_01x01, J202 Conn_01x01, J203 Conn_01x01, J204 Conn_01x01, J205 Conn_01x01, J206 Conn_01x01, J207 Conn_01x01, J208 Conn_01x01, J209 Conn_01x01, J210 Conn_01x01, J211 Conn_01x01, J212 Conn_01x01, J214 Conn_01x01, J215 Conn_01x01, J216 Conn_01x01, J217 Conn_01x01, J301 Conn_01x01, J302 Conn_01x01, J303 Conn_01x01, J304 Conn_01x01, J305 Conn_01x01, J306 Conn_01x01, J307 Conn_01x01, J308 Conn_01x01, J401 Conn_01x01, Q201 BD135, Q301 MMBT3904, Q302 MMBT3906, Q303 MMBT3904, Q401 MMBT3904, SW301 SW_Push, U201 ADR1000, U202 OPA2172, U301 L78L33_SOT89, U302 LT3439, U303 TMP117, U304 BR24H64FVM, U305 LT3045xMSE, U306 L78L33_SOT89, U307 L79L05_SOT89, U401 ADA4523, U402 ADG5401F, U403 ADA4523, U404 ADA4523, U405 D60V0L4B10LP

Commit message: Update adrmu6layer.kicad_pcb
Parts:
- moved R316 0.55 mm to (78.4, 64.5)
- moved SW301 0.28 mm to (73.3, 60.7)

Commit message: asdf
Parts:
- D308: value SMAJ15A-13-F -> SMAJ15A-18
- JP213: value Jumper_2_Open -> Jumper_2_Bridged
- R210: value 0 -> 62k
- R308: value 4k99 -> 2k7
- R406: value 4.99k -> 4k99
- moved J203 2.54 mm to (96.5, 109.2)
- turned JP213 to 0 degrees
Connections:
- JP213 pad 1: /Reference Circuit/J213_Pin1 -> /Reference Circuit/7Vref
- JP213 pad 2: /Reference Circuit/7Vref -> /Reference Circuit/J213_Pin1
Routing:
- net /Reference Circuit/JP201_Pin1: track 6.18 -> 5.13 mm
Changed lines of the file:
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@@
     (property "Sheetfile" "dcdc.kicad_sch")
     (property "Sheetname" "DC-DC converter")
-    (attr smd)
+    (property "exclude_from_bom" "")
+    (attr smd exclude_from_bom)
     (fp_text reference "R318" (at 3.8 0.05) (layer "F.SilkS")
       (effects (font (size 1 1) (thickness 0.15)))
@@
       (effects (font (size 0.7 0.7) (thickness 0.125)))
     )
-    (fp_text value "4.99k" (at 0 1.65) (layer "F.Fab")
+    (fp_text value "4k99" (at 0 1.65) (layer "F.Fab")
       (effects (font (size 1 1) (thickness 0.15)))
     )
@@
     (property "Sheetfile" "ref.kicad_sch")
     (property "Sheetname" "Reference Circuit")
-    (attr smd)
+    (property "exclude_from_bom" "")
+    (attr smd exclude_from_bom)
     (fp_text reference "R221" (at -0.55 -1.55) (layer "F.SilkS")
       (effects (font (size 1 1) (thickness 0.15)))
@@
   )
   (footprint "Connector_Wire:SolderWire-0.1sqmm_1x01_D0.4mm_OD1mm" (layer "F.Cu")
-    (at 93.98 109.22)
+    (at 96.52 109.22)
     (descr "Soldered wire connection, for a single 0.1 mm² wire, basic insulation, conductor diameter 0.4mm, outer diameter 1mm, size source Multi-Contact FLEXI-E 0.1 (https://ec.staubli.com/AcroFiles/Catalogues/TM_Cab-Main-11014119_(en)_hi.pdf), bend radius 3 times outer diameter, generated with kicad-footprint-generator")
     (tags "connector wire 0.1sqmm")
@@
       (effects (font (size 0.7 0.7) (thickness 0.125)))
     )
-    (fp_text value "4k99" (at 0 1.65 90) (layer "F.Fab")
+    (fp_text value "2k7" (at 0 1.65 90) (layer "F.Fab")
       (effects (font (size 1 1) (thickness 0.15)))
     )
@@
     (property "Sheetfile" "ref.kicad_sch")
     (property "Sheetname" "Reference Circuit")
-    (property "exclude_from_bom" "")
-    (attr smd exclude_from_bom)
+    (attr smd)
     (fp_text reference "R210" (at -0.061 2.736) (layer "F.SilkS") hide
       (effects (font (size 1 1) (thickness 0.15)))
     )
-    (fp_text value "0" (at 0 1.65) (layer "F.Fab")
+    (fp_text value "62k" (at 0 1.65) (layer "F.Fab")
       (effects (font (size 1 1) (thickness 0.15)))
     )
@@
       (effects (font (size 1 1) (thickness 0.15)))
     )
-    (fp_text value "SMAJ15A-13-F" (at 0 2.6) (layer "F.Fab")
+    (fp_text value "SMAJ15A-18" (at 0 2.6) (layer "F.Fab")
       (effects (font (size 1 1) (thickness 0.15)))
     )
@@
   )
   (footprint "Jumper:SolderJumper-2_P1.3mm_Open_RoundedPad1.0x1.5mm" (layer "B.Cu")
-    (at 94.650624 87.249 180)
+    (at 94.650624 87.249)
     (descr "SMD Solder Jumper, 1x1.5mm, rounded Pads, 0.3mm gap, open")
     (tags "solder jumper open")
@@
       (effects (font (size 1 1) (thickness 0.15)) (justify mirror))
     )
-    (fp_text value "Jumper_2_Open" (at 0 -1.9) (layer "B.Fab")
+    (fp_text value "Jumper_2_Bridged" (at 0 -1.9) (layer "B.Fab")
       (effects (font (size 1 1) (thickness 0.15)) (justify mirror))
     )
@@
     (fp_line (start 1.65 -1.25) (end 1.65 1.25) (layer "B.CrtYd") (width 0.05))
     (fp_line (start -1.65 1.25) (end 1.65 1.25) (layer "B.CrtYd") (width 0.05))
-    (pad "1" smd custom (at -0.65 0 180) (size 1 0.5) (layers "B.Cu" "B.Mask")
-      (net 128 "/Reference Circuit/J213_Pin1") (pinfunction "A") (pintype "passive") (zone_connect 2)
+    (pad "1" smd custom (at -0.65 0) (size 1 0.5) (layers "B.Cu" "B.Mask")
+      (net 21 "/Reference Circuit/7Vref") (pinfunction "A") (pintype "passive") (zone_connect 2)
       (options (clearance outline) (anchor rect))
       (primitives
@@
           ) (width 0) (fill yes))
       ))
-    (pad "2" smd custom (at 0.65 0 180) (size 1 0.5) (layers "B.Cu" "B.Mask")
-      (net 21 "/Reference Circuit/7Vref") (pinfunction "B") (pintype "passive") (zone_connect 2)
+    (pad "2" smd custom (at 0.65 0) (size 1 0.5) (layers "B.Cu" "B.Mask")
+      (net 128 "/Reference Circuit/J213_Pin1") (pinfunction "B") (pintype "passive") (zone_connect 2)
       (options (clearance outline) (anchor rect))
       (primitives
@@
       ))
   )
+  (gr_circle (center 119.499624 87.249) (end 120.399624 87.249) (layer "F.Cu") (width 1.9) (fill none))
   (gr_circle (center 119.499624 87.254) (end 120.399624 87.254) (layer "In1.Cu") (width 1.9) (fill none))
   (gr_circle (center 119.499624 87.249) (end 128.499624 87.249) (layer "In1.Cu") (width 4) (fill none))
@@
   (gr_line (start 173.7 136.5) (end 173.4 133.4) (layer "F.SilkS") (width 0.15))
   (gr_line (start 187.589069 109.693078) (end 184.444084 122.306922) (layer "F.SilkS") (width 0.15))
+  (gr_arc (start 127.499999 80.500001) (mid 111.97414 94.533395) (end 126.515786 79.482515) (layer "F.SilkS") (width 0.15))
   (gr_line (start 187.589069 109.693078) (end 187.205294 122.818683) (layer "F.SilkS") (width 0.15))
   (gr_line (start 190.008288 122.990121) (end 190 126.5) (layer "F.SilkS") (width 0.15))
@@
   (gr_line (start 198.25075 121.462471) (end 199.5 124.5) (layer "F.SilkS") (width 0.15))
   (gr_line (start 192.419219 90.297043) (end 192.802994 77.171438) (layer "F.SilkS") (width 0.15))
-  (gr_line (start 81.75 133.75) (end 82.25 133) (layer "F.SilkS") (width 0.15))
   (gr_line (start 190 77) (end 190 73.5) (layer "F.SilkS") (width 0.15))
   (gr_line (start 191.226981 109.915583) (end 192.811282 122.818683) (layer "F.SilkS") (width 0.15))
@@
   (gr_rect (start 70 50) (end 230 53) (layer "F.Mask") (width 0.15) (fill solid))
   (gr_circle (center 119.499624 87.249) (end 126.499624 87.249) (layer "F.Mask") (width 0.2) (fill solid))
+  (gr_line (start 93.98 93.98) (end 93.98 91.44) (layer "Dwgs.User") (width 0.15))
+  (gr_line (start 96.52 101.6) (end 93.98 104.14) (layer "Dwgs.User") (width 0.15))
+  (gr_line (start 96.52 96.52) (end 96.52 99.06) (layer "Dwgs.User") (width 0.15))
   (gr_line (start 230 53) (end 70 53) (layer "Dwgs.User") (width 0.15))
   (gr_line locked (start 230 147) (end 70 147) (layer "Dwgs.User") (width 0.15))
+  (gr_line (start 91.44 106.68) (end 91.44 109.22) (layer "Dwgs.User") (width 0.15))
+  (gr_line (start 93.98 96.52) (end 88.9 96.52) (layer "Dwgs.User") (width 0.15))
+  (gr_line (start 96.52 93.98) (end 96.52 96.52) (layer "Dwgs.User") (width 0.15))
+  (gr_line (start 91.44 106.68) (end 93.98 106.68) (layer "Dwgs.User") (width 0.15))
+  (gr_line (start 93.98 99.06) (end 93.98 101.6) (layer "Dwgs.User") (width 0.15))
+  (gr_line (start 93.98 104.14) (end 93.98 106.68) (layer "Dwgs.User") (width 0.15))
+  (gr_line (start 99.06 104.14) (end 99.06 109.22) (layer "Dwgs.User") (width 0.15))
   (gr_arc (start 172.32233 117.67767) (mid 172.32233 116.263456) (end 173.736544 116.263456) (layer "Edge.Cuts") (width 0.1))
   (gr_arc (start 139 120.5) (mid 138 119.5) (end 139 118.5) (layer "Edge.Cuts") (width 0.1))
@@
   (segment (start 99.06 96.52) (end 96.52 96.52) (width 2) (layer "B.Cu") (net 28))
   (segment (start 91.44 99.06) (end 93.98 99.06) (width 2) (layer "B.Cu") (net 29))
-  (segment (start 96.75 113) (end 96.75 111.99) (width 2) (layer "B.Cu") (net 30))
+  (segment (start 96.52 112.77) (end 96.52 109.22) (width 2) (layer "B.Cu") (net 30))
+  (segment (start 96.75 113) (end 96.52 112.77) (width 2) (layer "B.Cu") (net 30))
   (segment (start 96.75 113) (end 95.5 113) (width 1) (layer "B.Cu") (net 30))
-  (segment (start 96.75 111.99) (end 93.98 109.22) (width 2) (layer "B.Cu") (net 30))
   (segment (start 91.44 93.98) (end 93.98 93.98) (width 2) (layer "B.Cu") (net 31))
   (segment (start 93.98 96.52) (end 91.44 96.52) (width 2) (layer "B.Cu") (net 32))

Commit message: Rev. 1.0
Parts:
- removed JP201: Jumper_2_Open, Jumper:SolderJumper-2_P1.3mm_Open_RoundedPad1.0x1.5mm
- removed R411, R415: 0R, Resistor_SMD:R_0805_2012Metric
- added C415: 470n, Capacitor_SMD:C_1206_3216Metric, F.Cu at (125.8, 133.8)
- added C416: 100n 50V, Capacitor_SMD:C_0603_1608Metric, F.Cu at (132.8, 129.9)
- added C417: 100n 50V, Capacitor_SMD:C_0603_1608Metric, B.Cu at (146.1, 128.0)
- added C418: 22u 25V, Capacitor_SMD:C_1206_3216Metric, F.Cu at (134.9, 124.4)
- added C419: 100n 50V, Capacitor_SMD:C_0603_1608Metric, F.Cu at (151.6, 130.5)
- added C420: 1u, Capacitor_SMD:C_0805_2012Metric, F.Cu at (144.4, 122.3)
- added C421: 1u, Capacitor_SMD:C_0805_2012Metric, F.Cu at (172.0, 136.1)
- added JP410: Jumper_2_Bridged, Jumper:SolderJumper-2_P1.3mm_Bridged_RoundedPad1.0x1.5mm, F.Cu at (153.9, 128.2)
- added JP411: Jumper_2_Bridged, Jumper:SolderJumper-2_P1.3mm_Bridged_RoundedPad1.0x1.5mm, F.Cu at (151.3, 128.3)
- added RN202: DNP, Crystal:Resonator-3Pin_W10.0mm_H5.0mm, F.Cu at (104.1, 132.1)
- added RN402: DNP, Crystal:Resonator-3Pin_W10.0mm_H5.0mm, F.Cu at (140.8, 111.8)
- moved R301 5.03 mm to (197.7, 62.8), turned to -90 degrees
- moved C303 2.00 mm to (207.0, 58.3)
- moved R304 0.15 mm to (195.7, 62.8)
Routing:
- net /DC-DC converter/sync: track 45.1 -> 42.5 mm
- net /Buffer/JP404_pin2: track 109.2 -> 111.5 mm
- net /Buffer/GNDf: track 92.1 -> 93.9 mm
- net /Buffer/U403_-in: track 6.91 -> 8.65 mm
- net /Buffer/U403_out: track 14.6 -> 16.4 mm
- net /Buffer/U401_out: track 10.5 -> 12.2 mm
- net /Buffer/U401_-in: track 11.8 -> 13.5 mm
- net +12V: track 158.7 -> 160.2 mm
- net /Reference Circuit/ADR_Pin6: track 51.5 -> 50.2 mm
- net /Reference Circuit/JP201_Pin1: track 5.13 -> 3.88 mm
- net /Reference Circuit/ADR_Pin8: track 116.2 -> 115.2 mm
- net /Buffer/U402_DFB: track 7.54 -> 8.29 mm
- net /Buffer/U404_out: track 20.2 -> 19.6 mm
Other:
- board text added: "ADRmu 10V Standard Rev 1.0"
- board text removed: "ADRmu 10V Standard Rev 0.9"
