File: module_reference/adrmu6layer.kicad_pcb (KiCad board)
At the start: 6 copper layers, 160 x 100 mm, 226 parts, among them J101 Harting 09042326831, J102 OutHf, J103 OutHs, J104 7Vref, J105 Lo, J106 12VinC, J107 OutLs, J108 OutLf, J201 Conn_01x01, J202 Conn_01x01, J203 Conn_01x01, J204 Conn_01x01, J205 Conn_01x01, J206 Conn_01x01, J207 Conn_01x01, J208 Conn_01x01, J209 Conn_01x01, J210 Conn_01x01, J211 Conn_01x01, J212 Conn_01x01, J214 Conn_01x01, J215 Conn_01x01, J216 Conn_01x01, J217 Conn_01x01, J301 Conn_01x01, J302 Conn_01x01, J303 Conn_01x01, J304 Conn_01x01, J305 Conn_01x01, J306 Conn_01x01, J307 Conn_01x01, J308 Conn_01x01, J401 Conn_01x01, Q201 BD135, Q301 MMBT3904, Q302 MMBT3906, Q303 MMBT3904, Q401 MMBT3904, SW301 SW_Push, U201 ADR1000, U202 OPA2172, U301 L78L33_SOT89, U302 LT3439, U303 TMP117, U304 BR24H64FVM, U305 LT3045xMSE, U306 L78L33_SOT89, U307 L79L05_SOT89, U401 ADA4523, U402 ADG5401F, U403 ADA4523, U404 ADA4523, U405 D60V0L4B10LP

Commit message: corrected noise measurements
Parts:
- added D401: 1N4148, Diode_SMD:D_SOD-123, F.Cu at (159.1, 120.1)
- added R411: 1k, Resistor_SMD:R_0805_2012Metric, F.Cu at (151.3, 121.8)
- added R415: 10k, Resistor_SMD:R_0805_2012Metric, F.Cu at (148.2, 124.7)
- JP213: footprint Jumper:SolderJumper-2_P1.3mm_Open_RoundedPad1.0x1.5mm -> Jumper:SolderJumper-2_P1.3mm_Bridged_RoundedPad1.0x1.5mm
- R406: value 4k99 -> 10k
- moved R406 3.50 mm to (147.3, 122.0)
- moved J307 2.84 mm to (128.2, 129.6)
- moved C412 2.05 mm to (143.6, 123.5)
- moved C420 2.05 mm to (142.4, 122.3)
- moved R409 1.86 mm to (146.1, 124.7)
- moved R309 1.00 mm to (157.9, 123.1)
- moved C404 0.91 mm to (134.0, 122.0)
- moved C418 0.91 mm to (134.0, 124.5)
- turned Q401 to -90 degrees
Connections:
- Q401 pad 1: /Buffer/OutLf -> Net-(Q401-Pad1)
- Q401 pad 3: /Buffer/U402_in -> Net-(Q401-Pad3)
Routing:
- net /Buffer/U402_in: track 4.82 -> 14.8 mm
- net /Buffer/OutLf: track 87.2 -> 94.7 mm, vias 1 -> 0
- net /Buffer/3Vf: track 19.0 -> 26.4 mm, vias 0 -> 2
- net Net-(Q401-Pad1): track 0.00 -> 6.77 mm
- net Net-(Q401-Pad3): track 0.00 -> 4.07 mm
- net /Buffer/U403_out: track 16.4 -> 19.8 mm
- net /Buffer/GNDf: track 93.9 -> 97.3 mm
- net /Buffer/-5Vf: track 59.7 -> 62.1 mm
- net /Buffer/FF: track 84.1 -> 85.2 mm
