File: module_reference/adrmu6layer.kicad_sch (KiCad schematic)
At the start: 13 parts, among them J101 Harting 09042326831, J102 OutHf, J103 OutHs, J104 7Vref, J105 Lo, J106 12VinC, J107 OutLs, J108 OutLf

Commit message: Rev 1.1 & Kicad 7 update
Parts:
- J106: footprint Connector_Wire:SolderWire-1sqmm_1x01_D1.4mm_OD2.7mm -> Connector_Wire:SolderWire-0.5sqmm_1x01_D0.9mm_OD2.3mm
