File: module_reference/dcdc.kicad_sch (KiCad schematic)
At the start: 59 parts, among them J301 Conn_01x01, J302 Conn_01x01, J303 Conn_01x01, J304 Conn_01x01, J305 Conn_01x01, Q301 MMBT3904, T301 Feryster RTN-40x25x15(M-083), U301 L78L33_SOT89, U302 LT3439, U303 TMP117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

Commit message: Ref module Rev. 0.9
Parts:
- added C314, C315, C317, C318: 100n 50V, Capacitor_SMD:C_0603_1608Metric, symbol Device:C
- added C316: 22u 25V, Capacitor_SMD:C_1206_3216Metric, symbol Device:C
- added D102, D103, D307: PMEG6010CEH, Diode_SMD:D_SOD-123F, symbol Device:D_Schottky
- added D308: SMAJ15A-13-F, Diode_SMD:D_SMA, symbol Device:D_Zener
- added F301: SF-0603S040-2, Fuse:Fuse_0603_1608Metric, symbol Device:Fuse
- added J306, J307: Conn_01x01, Connector_Wire:SolderWirePad_1x01_SMD_1x2mm, symbol Connector_Generic:Conn_01x01
- added J308: Conn_01x01, Connector_Wire:SolderWire-1sqmm_1x01_D1.4mm_OD3.9mm, symbol Connector_Generic:Conn_01x01
- added Q302: MMBT3906, Package_TO_SOT_SMD:SOT-23, symbol Transistor_BJT:MMBT3906
- added Q303: MMBT3904, Package_TO_SOT_SMD:SOT-23, symbol Transistor_BJT:MMBT3904
- added R314, R315, R316, R317: 10k, Resistor_SMD:R_0805_2012Metric, symbol Device:R
- added R318: DNP, Resistor_SMD:R_0805_2012Metric, symbol Device:R
- added SW301: SW_Push, Button_Switch_THT:SW_Tactile_SPST_Angled_PTS645Vx31-2LFS, symbol Switch:SW_Push
- added U306: L78L33_SOT89, Package_TO_SOT_SMD:SOT-89-3, symbol Regulator_Linear:L78L33_SOT89
- added U307: L79L05_SOT89, Package_TO_SOT_SMD:SOT-89-3, symbol Regulator_Linear:L79L05_SOT89
- C301, C302, C308, C309, C310, C311: footprint Capacitor_SMD:C_0805_2012Metric -> Capacitor_SMD:C_0603_1608Metric
- R303: value 49k9 -> 49.9k
- R308: value 49k9 -> 4k99
- R311: value 110k -> 130k
- R312: value 1M -> 750k
- R313: value 30k -> 18k
Connections:
- net +12V: now also D102.1 (K), D103.1 (K), Q302.2 (E), R317.1, SW301.2; no longer R303.1
- net 12Vf: now also C314.1, D307.1 (K), U306.3 (IN)
- net GND: now also C318.2, Q303.2 (E), R318.1
- net rectified+: now also F301.1; no longer C307.1, C309.1, Q301.3 (C), R309.2, U305.1 (IN), U305.2 (IN), U305.3 (IN), U305.4 (EN/UV)
- net xformer_B: now also J308.1 (Pin_1); no longer J305.1 (Pin_1)
- net GNDA renamed GNDf
- net GNDf: now also J305.1 (Pin_1), C314.2, C315.2, C316.1, C317.1, D308.2 (A), J307.1 (Pin_1), U306.2 (GND), U307.1 (GND); no longer D303.2 (A), D305.2 (A)
- net pwr_LED renamed D301_A
- net D301_A: now also R303.1; no longer R303.2
- net status renamed Q301_e
- net status_LED renamed D306_A
- new net +12VinA: D102.2 (A)
- new net +12VinB: D103.2 (A)
- new net +12VinC: D307.2 (A)
- new net -5Vf: C317.2, U307.3 (VO)
- new net 3Vf: C315.1, Q301.3 (C), R309.2, U306.1 (OUT)
- new net Q302_b: Q302.1 (B), R316.2
- new net Q302_c: Q302.3 (C), R303.2, R315.2
- new net Q303_b: C318.1, Q303.1 (B), R314.2, R315.1, R318.2
- new net Q303_c: Q303.3 (C), R316.1, R317.2
- new net SW301: R314.1, SW301.1
- new net U305_in: C307.1, C309.1, D308.1 (K), F301.2, J306.1 (Pin_1), U305.1 (IN), U305.2 (IN), U305.3 (IN), U305.4 (EN/UV)
- new net U307_vi: C316.2, D303.2 (A), D305.2 (A), U307.2 (VI)
Other:
- moved on the sheet: C303, C307, C310, C311, C312, C313, D301, D306, H301, H302, H303, H304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

Commit message: asdf
Parts:
- D308: value SMAJ15A-13-F -> SMAJ15A-18
- R308: value 4k99 -> 2k7
- R318: now left out of the parts list
Changed lines of the file:
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@@
       (effects (font (size 1.27 1.27)) (justify left))
     )
-    (property "Value" "SMAJ15A-13-F" (id 1) (at 171.45 45.7199 90)
+    (property "Value" "SMAJ15A-18" (id 1) (at 171.45 45.7199 90)
       (effects (font (size 1.27 1.27)) (justify left))
     )
@@
   )
   (symbol (lib_id "Device:R") (at 100.33 113.03 180) (unit 1)
-    (in_bom yes) (on_board yes) (fields_autoplaced)
+    (in_bom no) (on_board yes) (fields_autoplaced)
     (property "Reference" "R318" (id 0) (at 102.87 111.7599 0)
       (effects (font (size 1.27 1.27)) (justify right))
@@
     (in_bom yes) (on_board yes) (fields_autoplaced)
     (property "Reference" "R308" (id 0) (at 255.27 102.87 90))
-    (property "Value" "4k99" (id 1) (at 255.27 105.41 90))
+    (property "Value" "2k7" (id 1) (at 255.27 105.41 90))
     (property "Footprint" "Resistor_SMD:R_0805_2012Metric" (id 2) (at 255.27 100.838 90)
       (effects (font (size 1.27 1.27)) hide)

Commit message: Rev 1.1 & Kicad 7 update
Parts:
- removed U301, U306: L78L33_SOT89, Package_TO_SOT_SMD:SOT-89-3, symbol Regulator_Linear:L78L33_SOT89
- removed U304: BR24H64FVM, Package_SO:MSOP-8_3x3mm_P0.65mm, symbol Memory_EEPROM:24LC02
- added FL301: SRF0905A-472Y, Filter:Filter_Bourns_SRF0905_6.0x9.2mm, symbol Device:Filter_EMI_CommonMode
- added J309, J310: Conn_01x01, Connector_Wire:SolderWire-0.5sqmm_1x01_D0.9mm_OD2.3mm, symbol Connector_Generic:Conn_01x01
- added JP308, JP309, JP310: Jumper_2_Open, Jumper:SolderJumper-2_P1.3mm_Open_RoundedPad1.0x1.5mm, symbol Jumper:Jumper_2_Open
- added L301: 47µH, Inductor_SMD:L_Sunlord_SWPA3012S, symbol Device:L
- added U301, U306: HT75xx-1-SOT89, Package_TO_SOT_SMD:SOT-89-3, symbol Regulator_Linear:HT75xx-1-SOT89
- added U304: CAT24C256, Package_SO:SOIC-8_3.9x4.9mm_P1.27mm, symbol Memory_EEPROM:CAT24C256
- C305: value 22u 25V -> 100n 50V; footprint Capacitor_SMD:C_1206_3216Metric -> Capacitor_SMD:C_0603_1608Metric
- D302, D303, D304, D305, D307: footprint Diode_SMD:D_SOD-123F -> Diode_SMD:D_SOD-123
- D309: renamed from D102; footprint Diode_SMD:D_SOD-123F -> Diode_SMD:D_SOD-123
- D310: renamed from D103; footprint Diode_SMD:D_SOD-123F -> Diode_SMD:D_SOD-123
- J301, J302, J303, J304, J305, J308: footprint Connector_Wire:SolderWire-1sqmm_1x01_D1.4mm_OD3.9mm -> Connector_Wire:SolderWire-0.5sqmm_1x01_D0.9mm_OD2.3mm
Connections:
- net +12V: now also JP308.1 (A), L301.1, U301.2 (VIN); no longer C301.1, C306.1, J302.1 (Pin_1), U302.11 (~{SHDN}), U302.13 (VIN)
- net +3V3: now also U301.3 (VOUT), U304.8 (VCC)
- net 12Vf: now also U306.2 (VIN)
- net 3Vf: now also U306.3 (VOUT)
- net GND: now also U301.1 (GND), U304.4 (GND), U304.7 (WP)
- net GNDf: now also J310.1 (Pin_1), U306.1 (GND)
- net SCL: now also U304.6 (SCL)
- net SDA: now also U304.5 (SDA)
- net U304_a0: now also U304.1 (A0)
- net U304_a1: now also U304.2 (A1)
- net U304_a2: now also U304.3 (A2)
- net U305_in: now also FL301.2, JP309.2 (B); no longer F301.2
- net U307_vi: now also FL301.4, JP310.2 (B); no longer D303.2 (A), D305.2 (A)
- new net: F301.2, FL301.1, JP309.1 (A)
- new net: D303.2 (A), D305.2 (A), FL301.3, JP310.1 (A)
- new net U302_vin: C301.1, C306.1, J302.1 (Pin_1), J309.1 (Pin_1), JP308.2 (B), L301.2, U302.11 (~{SHDN}), U302.13 (VIN)
Other:
- moved on the sheet: C301, C307, C309, C310, C311, C312, C313, C314, C315, C316, C317, D306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

Commit message: Rev 1.2
Parts:
- removed FL301: SRF0905A-472Y, Filter:Filter_Bourns_SRF0905_6.0x9.2mm, symbol Device:Filter_EMI_CommonMode
- added FL301: Filter_EMI_LL_1423, Filter:Filter_Bourns_SRF0905_6.0x9.2mm, symbol Device:Filter_EMI_LL_1423
Connections:
- net U305_in: now also FL301.3
- net U307_vi: now also FL301.4
- net at F301.2, JP309.1 (A): now also FL301.2
- net at D303.2 (A), D305.2 (A), JP310.1 (A): now also FL301.1
Changed lines of the file:
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@@
   (title_block
     (title "DC-DC converter & misc")
-    (date "2023-02-15")
-    (rev "1.1")
+    (date "2023-03-08")
+    (rev "1.2")
     (company "RPG")
     (comment 1 "All resistors 0.1% MF unless otherwise noted")
@@
   (junction (at 83.82 83.82) (diameter 0) (color 0 0 0 0)
   )
+  (junction (at 161.29 40.64) (diameter 0) (color 0 0 0 0)
+  )
   (junction (at 93.98 153.67) (diameter 0) (color 0 0 0 0)
   )
@@
   (junction (at 50.8 29.21) (diameter 0) (color 0 0 0 0)
   )
-  (junction (at 161.29 40.64) (diameter 0) (color 0 0 0 0)
-  )
   (junction (at 257.81 60.96) (diameter 0) (color 0 0 0 0)
   )
@@
     )
   )
+  (symbol (lib_id "Device:Filter_EMI_LL_1423") (at 166.37 38.1 0) (unit 1)
+    (in_bom yes) (on_board yes) (dnp no) (fields_autoplaced)
+    (property "Reference" "FL301" (at 165.989 31.75 0)
+      (effects (font (size 1.27 1.27)))
+    )
+    (property "Value" "Filter_EMI_LL_1423" (at 165.989 34.29 0)
+      (effects (font (size 1.27 1.27)))
+    )
+    (property "Footprint" "Filter:Filter_Bourns_SRF0905_6.0x9.2mm" (at 166.37 44.45 0)
+      (effects (font (size 1.27 1.27)) hide)
+    )
+    (property "Datasheet" "https://datasheet.lcsc.com/lcsc/1809291820_BOURNS-SRF0905A-472Y_C113524.pdf" (at 166.37 37.084 90)
+      (effects (font (size 1.27 1.27)) hide)
+    )
+    (pin "1")
+    (pin "2")
+    (pin "3")
+    (pin "4")
+    (instances
+      (project "adrmu6layer"
+        (path "/e63e39d7-6ac0-4ffd-8aa3-1841a4541b55/b2eac6f7-6f2b-41aa-9eec-9c2e749d1013"
+          (reference "FL301") (unit 1)
+        )
+      )
+    )
+  )
   (symbol (lib_id "power:+3V3") (at 163.83 90.17 0) (unit 1)
     (in_bom yes) (on_board yes) (dnp no) (fields_autoplaced)
@@
         )
       )
-    )
-  )
-  (symbol (lib_id "Device:Filter_EMI_CommonMode") (at 166.37 38.1 0) (unit 1)
-    (in_bom yes) (on_board yes) (dnp no)
-    (property "Reference" "FL301" (at 167.64 29.21 0)
-      (effects (font (size 1.27 1.27)))
-    )
-    (property "Value" "SRF0905A-472Y" (at 166.37 25.4 0)
-      (effects (font (size 1.27 1.27)))
-    )
-    (property "Footprint" "Filter:Filter_Bourns_SRF0905_6.0x9.2mm" (at 166.37 37.084 0)
-      (effects (font (size 1.27 1.27)) hide)
-    )
-    (property "Datasheet" "~" (at 166.37 37.084 0)
-      (effects (font (size 1.27 1.27)) hide)
-    )
-    (pin "1")
-    (pin "2")
-    (pin "3")
-    (pin "4")
-    (instances
-      (project "adrmu6layer"
-        (path "/e63e39d7-6ac0-4ffd-8aa3-1841a4541b55/b2eac6f7-6f2b-41aa-9eec-9c2e749d1013"
-          (reference "FL301") (unit 1)
-        )
-      )
