File: module_reference/ref.kicad_sch (KiCad schematic)
At the start: 77 parts, among them J201 Conn_01x01, J202 Conn_01x01, J203 Conn_01x01, J204 Conn_01x01, J205 Conn_01x01, J206 Conn_01x01, J207 Conn_01x01, J208 Conn_01x01, J209 Conn_01x01, J210 Conn_01x01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

Commit message: Rev. 1.0
Parts:
- removed JP201: Jumper_2_Open, Jumper:SolderJumper-2_P1.3mm_Open_RoundedPad1.0x1.5mm, symbol Jumper:Jumper_2_Open
- added RN202: DNP, Crystal:Resonator-3Pin_W10.0mm_H5.0mm, symbol Device:VoltageDivider
Connections:
- net 7Vref: now also RN202.1
- net ADR_Pin6: now also RN202.2
- net ADR_Pin7: now also RN202.3
Changed lines of the file:
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@@
   (title_block
     (title "Reference circuit")
-    (date "2022-12-26")
-    (rev "0.9")
+    (date "2023-01-29")
+    (rev "1.0")
     (company "RPG")
     (comment 1 "All resistors 0.1% MF unless otherwise noted")
@@
     (stroke (width 0) (type default) (color 0 0 0 0))
   )
+  (wire (pts (xy 109.22 175.26) (xy 110.49 175.26))
+    (stroke (width 0) (type default) (color 0 0 0 0))
+  )
   (wire (pts (xy 191.77 55.88) (xy 194.31 55.88))
     (stroke (width 0) (type default) (color 0 0 0 0))
@@
     (stroke (width 0) (type default) (color 0 0 0 0))
   )
-  (wire (pts (xy 124.46 143.51) (xy 125.73 143.51))
-    (stroke (width 0) (type default) (color 0 0 0 0))
-  )
   (wire (pts (xy 265.43 133.35) (xy 265.43 135.89))
     (stroke (width 0) (type default) (color 0 0 0 0))
@@
     (stroke (width 0) (type default) (color 0 0 0 0))
   )
-  (wire (pts (xy 113.03 143.51) (xy 114.3 143.51))
-    (stroke (width 0) (type default) (color 0 0 0 0))
-  )
   (wire (pts (xy 147.32 120.65) (xy 149.86 120.65))
     (stroke (width 0) (type default) (color 0 0 0 0))
@@
     (stroke (width 0) (type default) (color 0 0 0 0))
   )
+  (wire (pts (xy 105.41 168.91) (xy 105.41 167.64))
+    (stroke (width 0) (type default) (color 0 0 0 0))
+  )
   (wire (pts (xy 182.88 27.94) (xy 185.42 27.94))
     (stroke (width 0) (type default) (color 0 0 0 0))
   )
   (wire (pts (xy 223.52 161.29) (xy 232.41 161.29))
+    (stroke (width 0) (type default) (color 0 0 0 0))
+  )
+  (wire (pts (xy 105.41 182.88) (xy 105.41 181.61))
     (stroke (width 0) (type default) (color 0 0 0 0))
   )
@@
     (effects (font (size 0.635 0.635)) (justify left bottom))
   )
+  (label "ADR_Pin7" (at 105.41 182.88 180)
+    (effects (font (size 1.27 1.27)) (justify right bottom))
+  )
   (label "U202B_-in" (at 125.73 69.85 180)
     (effects (font (size 0.5 0.5)) (justify right bottom))
@@
     (effects (font (size 0.5 0.5)) (justify right bottom))
   )
+  (label "ADR_Pin6" (at 110.49 175.26 0)
+    (effects (font (size 1.27 1.27)) (justify left bottom))
+  )
   (label "7Vref" (at 24.13 132.08 180)
     (effects (font (size 1.27 1.27)) (justify right bottom))
@@
   (label "ADR_Pin7" (at 195.58 151.13 0)
     (effects (font (size 1.27 1.27)) (justify left bottom))
+  )
+  (label "7Vref" (at 105.41 167.64 180)
+    (effects (font (size 1.27 1.27)) (justify right bottom))
   )
   (label "RN203_Pin4" (at 144.78 109.22 0)
@@
     (pin "1")
   )
+  (symbol (lib_id "Device:VoltageDivider") (at 105.41 175.26 0) (unit 1)
+    (in_bom no) (on_board yes) (fields_autoplaced)
+    (property "Reference" "RN202" (id 0) (at 102.87 173.9899 0)
+      (effects (font (size 1.27 1.27)) (justify right))
+    )
+    (property "Value" "DNP" (id 1) (at 102.87 176.5299 0)
+      (effects (font (size 1.27 1.27)) (justify right))
+    )
+    (property "Footprint" "Crystal:Resonator-3Pin_W10.0mm_H5.0mm" (id 2) (at 117.475 175.26 90)
+      (effects (font (size 1.27 1.27)) hide)
+    )
+    (property "Datasheet" "https://xdevs.com/doc/VPG/vhd200_144.pdf" (id 3) (at 110.49 175.26 0)
+      (effects (font (size 1.27 1.27)) hide)
+    )
+    (pin "1")
+    (pin "2")
+    (pin "3")
+  )
   (symbol (lib_id "ADRmu_Library:Vishay TDP") (at 34.29 132.08 90) (unit 1)
     (in_bom no) (on_board yes) (fields_autoplaced)
@@
       (effects (font (size 1.27 1.27)) hide)
     )
-    (pin "1")
-    (pin "2")
-  )
-  (symbol (lib_id "Jumper:Jumper_2_Open") (at 119.38 143.51 0) (unit 1)
-    (in_bom no) (on_board yes)
-    (property "Reference" "JP201" (id 0) (at 118.11 151.13 0)
-      (effects (font (size 1.27 1.27)) (justify left))
-    )
-    (property "Value" "Jumper_2_Open" (id 1) (at 120.6499 140.97 90)
-      (effects (font (size 1.27 1.27)) (justify left) hide)
-    )
-    (property "Footprint" "Jumper:SolderJumper-2_P1.3mm_Open_RoundedPad1.0x1.5mm" (id 2) (at 119.38 143.51 0)
-      (effects (font (size 1.27 1.27)) hide)
-    )
-    (property "Datasheet" "~" (id 3) (at 119.38 143.51 0)
-      (effects (font (size 1.27 1.27)) hide)
-    )

Commit message: Rev 1.2
Parts:
- added J213: Conn_01x01, Connector_Wire:SolderWire-0.1sqmm_1x01_D0.4mm_OD1mm, symbol Connector_Generic:Conn_01x01
Connections:
- net ADR_Pin7: now also J213.1 (Pin_1)
Changed lines of the file:
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@@
   (title_block
     (title "Reference circuit")
-    (date "2023-02-15")
-    (rev "1.1")
+    (date "2023-03-08")
+    (rev "1.2")
     (company "RPG")
     (comment 1 "All resistors 0.1% MF unless otherwise noted")
@@
   (junction (at 125.73 143.51) (diameter 0) (color 0 0 0 0)
   )
+  (junction (at 115.57 156.21) (diameter 0) (color 0 0 0 0)
+  )
   (junction (at 180.34 44.45) (diameter 0) (color 0 0 0 0)
   )
@@
     (stroke (width 0) (type default))
   )
+  (wire (pts (xy 115.57 156.21) (xy 115.57 158.75))
+    (stroke (width 0) (type default))
+  )
   (wire (pts (xy 130.81 158.75) (xy 130.81 156.21))
     (stroke (width 0) (type default))
@@
     (stroke (width 0) (type default))
   )
+  (wire (pts (xy 115.57 156.21) (xy 120.65 156.21))
+    (stroke (width 0) (type default))
+  )
   (wire (pts (xy 165.1 120.65) (xy 168.91 120.65))
     (stroke (width 0) (type default))
@@
     (stroke (width 0) (type default))
   )
-  (wire (pts (xy 113.03 156.21) (xy 120.65 156.21))
+  (wire (pts (xy 113.03 156.21) (xy 115.57 156.21))
     (stroke (width 0) (type default))
   )
@@
   (symbol (lib_id "Connector_Generic:Conn_01x01") (at 120.65 163.83 270) (unit 1)
     (in_bom no) (on_board yes) (dnp no) (fields_autoplaced)
-    (property "Reference" "J216" (at 123.19 162.5599 90)
+    (property "Reference" "J216" (at 123.19 163.195 90)
       (effects (font (size 1.27 1.27)) (justify left))
     )
-    (property "Value" "Conn_01x01" (at 123.19 165.0999 90)
+    (property "Value" "Conn_01x01" (at 123.19 165.735 90)
       (effects (font (size 1.27 1.27)) (justify left))
     )
@@
         )
       )
+    )
+  )
+  (symbol (lib_id "Connector_Generic:Conn_01x01") (at 115.57 163.83 270) (unit 1)
+    (in_bom no) (on_board yes) (dnp no) (fields_autoplaced)
+    (property "Reference" "J213" (at 115.57 167.64 90)
+      (effects (font (size 1.27 1.27)))
+    )
+    (property "Value" "Conn_01x01" (at 115.57 170.18 90)
+      (effects (font (size 1.27 1.27)))
+    )
+    (property "Footprint" "Connector_Wire:SolderWire-0.1sqmm_1x01_D0.4mm_OD1mm" (at 115.57 163.83 0)
+      (effects (font (size 1.27 1.27)) hide)
+    )
+    (property "Datasheet" "~" (at 115.57 163.83 0)
+      (effects (font (size 1.27 1.27)) hide)
+    )
+    (pin "1")
+    (instances
+      (project "adrmu6layer"
+        (path "/e63e39d7-6ac0-4ffd-8aa3-1841a4541b55/027929a1-62dd-40f4-83d4-39d0de3b1543"
+          (reference "J213") (unit 1)
+        )
+      )
