File: resistor_network/resistor_network.kicad_sch (KiCad schematic)
At the start: 26 parts, among them J1 Vin_reg, J2 GND, J3 Vin_pow, J4 Conn_01x08, J5 Conn_01x08, Q1 BC847, Q2 BCX53

Commit message: New backplane, Reference Rev 0.6 with heated resistor network support
Connections:
- net at J2.1 (Pin_1), Q1.2 (E), TH1.2: now also Q2.2 (C); no longer Q2.3 (E)
- net at R10.2, R3.2, R4.1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: now also Q2.3 (E); no longer Q2.2 (C)
Changed lines of the file:
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@@
     (pin "8")
   )
-  (symbol (lib_id "Transistor_BJT:BCX53") (at 115.57 99.06 0) (unit 1)
+  (symbol (lib_id "Transistor_BJT:BCX53") (at 115.57 99.06 0) (mirror x) (unit 1)
     (in_bom yes) (on_board yes) (fields_autoplaced)
     (property "Reference" "Q2" (id 0) (at 120.65 97.7899 0)
@@
       (effects (font (size 1.27 1.27)) (justify left))
     )
-    (property "Footprint" "Package_TO_SOT_SMD:SOT-89-3" (id 2) (at 120.65 100.965 0)
+    (property "Footprint" "Package_TO_SOT_SMD:SOT-89-3" (id 2) (at 120.65 97.155 0)
       (effects (font (size 1.27 1.27) italic) (justify left) hide)
     )
