File: backplane/backplane.kicad_pcb (KiCad board)
At the start: 2 copper layers, 425.3 x 128.7 mm, 28 parts, among them J101 DIN41612_02x16_AC_EvenPins, J102 DIN41612_02x16_AC_EvenPins, J103 DIN41612_02x16_AC_EvenPins, J104 DIN41612_02x16_AC_EvenPins, J105 DIN41612_02x16_AC_EvenPins, J106 DIN41612_02x16_AC_EvenPins, J107 DIN41612_02x16_AC_EvenPins, J108 DIN41612_02x16_AC_EvenPins, J109 Conn_01x03, J110 Conn_01x03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

Commit message: Rev 0.2 Backplane
Parts:
- added JP105: Jumper_2_Open, Jumper:SolderJumper-2_P1.3mm_Open_RoundedPad1.0x1.5mm, B.Cu at (406.8, 61.6)
- J110: footprint Connector_JST:JST_PH_B3B-PH-K_1x03_P2.00mm_Vertical -> Connector_JST:JST_XH_B3B-XH-A_1x03_P2.50mm_Vertical
- moved J109 10.6 mm to (405.3, 79.0), turned to 90 degrees
Connections:
- J101 pad a4: Net-(J101-Pada4) -> Net-(J110-Pad3)
- J101 pad c4: Net-(J101-Pada4) -> Net-(J110-Pad3)
- J102 pad a4: Net-(J101-Pada4) -> Net-(J110-Pad3)
- J102 pad c4: Net-(J101-Pada4) -> Net-(J110-Pad3)
- J103 pad a4: Net-(J103-Pada4) -> Net-(J110-Pad3)
- J103 pad c4: Net-(J103-Pada4) -> Net-(J110-Pad3)
- J104 pad a4: Net-(J103-Pada4) -> Net-(J110-Pad3)
- J104 pad c4: Net-(J103-Pada4) -> Net-(J110-Pad3)
- J105 pad a4: Net-(J105-Pada4) -> Net-(J110-Pad3)
- J105 pad c4: Net-(J105-Pada4) -> Net-(J110-Pad3)
- J106 pad a4: Net-(J105-Pada4) -> Net-(J110-Pad3)
- J106 pad c4: Net-(J105-Pada4) -> Net-(J110-Pad3)
- J107 pad a4: Net-(J107-Pada4) -> Net-(J110-Pad3)
- J107 pad c4: Net-(J107-Pada4) -> Net-(J110-Pad3)
- J108 pad a4: Net-(J107-Pada4) -> Net-(J110-Pad3)
- J108 pad c4: Net-(J107-Pada4) -> Net-(J110-Pad3)
- J109 pad 1: Net-(J102-Pada20) -> Earth_Protective
- J109 pad 3: Earth_Protective -> Net-(J102-Pada20)
- J110 pad 3: Earth_Protective -> Net-(J110-Pad3)
Routing:
- net Net-(J110-Pad3): track 0.00 -> 415.8 mm
- net Net-(J107-Pada4): track 66.0 -> 0.00 mm
- net Net-(J101-Pada4): track 66.0 -> 0.00 mm
- net Net-(J105-Pada4): track 66.0 -> 0.00 mm
- net Net-(J103-Pada4): track 66.0 -> 0.00 mm
- net Net-(J102-Pada22): track 336.7 -> 341.0 mm
- net Net-(J102-Pada20): track 336.6 -> 341.0 mm
Other:
- board text added: "+ - PE"
