File: backplane/backplane.kicad_sch (KiCad schematic)
At the start: 28 parts, among them J101 DIN41612_02x16_AC_EvenPins, J102 DIN41612_02x16_AC_EvenPins, J103 DIN41612_02x16_AC_EvenPins, J104 DIN41612_02x16_AC_EvenPins, J105 DIN41612_02x16_AC_EvenPins, J106 DIN41612_02x16_AC_EvenPins, J107 DIN41612_02x16_AC_EvenPins, J108 DIN41612_02x16_AC_EvenPins, J109 Conn_01x03, J110 Conn_01x03, J111 Conn_01x01, J112 Conn_01x01

Commit message: Rev 0.2 Backplane
Parts:
- added JP105: Jumper_2_Open, Jumper:SolderJumper-2_P1.3mm_Open_RoundedPad1.0x1.5mm, symbol Jumper:Jumper_2_Open
- J110: footprint Connector_JST:JST_PH_B3B-PH-K_1x03_P2.00mm_Vertical -> Connector_JST:JST_XH_B3B-XH-A_1x03_P2.50mm_Vertical
Connections:
- net Earth_Protective: now also J109.1 (Pin_1), JP105.1 (A); no longer J109.3 (Pin_3), J110.3 (Pin_3)
- net at J102.a20 (Pin_a20), J102.c20 (Pin_c20), J104.a20 (Pin_a20)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: now also J109.3 (Pin_3); no longer J109.1 (Pin_1)
- net at J107.a4 (Pin_a4), J107.c4 (Pin_c4), J108.a4 (Pin_a4)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: now also J101.a4 (Pin_a4), J101.c4 (Pin_c4), J102.a4 (Pin_a4), J102.c4 (Pin_c4), J103.a4 (Pin_a4), J103.c4 (Pin_c4), J104.a4 (Pin_a4), J104.c4 (Pin_c4), J105.a4 (Pin_a4), J105.c4 (Pin_c4), J106.a4 (Pin_a4), J106.c4 (Pin_c4), J110.3 (Pin_3), JP105.2 (B)

Commit message: Update backplane.kicad_sch
Parts:
- added D? (x4): D, Diode_THT:D_A-405_P12.70mm_Horizontal, symbol Device:D
- JP105: footprint Jumper:SolderJumper-2_P1.3mm_Open_RoundedPad1.0x1.5mm -> Jumper:SolderJumper-2_P1.3mm_Bridged_RoundedPad1.0x1.5mm
Connections:
- net at J107.a2 (Pin_a2), J107.c2 (Pin_c2), J108.a2 (Pin_a2)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: now also D?.1 (K), D?.2 (A)
- net at J105.a2 (Pin_a2), J105.c2 (Pin_c2), J106.a2 (Pin_a2)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: now also D?.1 (K), D?.2 (A)
- net at J103.a2 (Pin_a2), J103.c2 (Pin_c2), J104.a2 (Pin_a2)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: now also D?.1 (K), D?.2 (A)
- net at J101.a2 (Pin_a2), J101.c2 (Pin_c2), J102.a2 (Pin_a2)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: now also D?.1 (K), D?.2 (A)
